File: Z80-FPGA-SBC/SBC.sch (KiCad schematic (older format))
At the start: 157 parts, among them J1 USB_2, K1 CONN_3, K12 CONN_3, K6 CONN_3, K8 CONN_3, K9 CONN_3, P1 PARALLEL, P10 PROG_B, P14 CONN_6, P17 CONN_1, P18 CONN_1, P2 CLK_CPU, P21 S100_MALE, P4 XILINX CABLE, P5 CLK_UART, P6 RESET, P7 CPLD_JTAG, P8 PF_JTAG, P9 S6_JTAG, Q1 ^^NPN-BC817-SOT323, SW1 SW_PUSH, SW3 PROG_B, U1 16550, U10 LM1086CS, U11 LF25CDT, U12 LD1117DT12, U13 74LS245, U14 74LS245, U15 74LS245, U16 27C080, U17 POWER_SELECT, U19 8255, U2 27C080, U22 74LS541, U24 Z80-CPU, U25 IS61LV5128AL-SOJ32, U26 74LS06N, U27 IS61LV5128AL-SOJ32, U28 FT232R, U3 23LC1024, U30 XC6SLX9-TQ144, U31 CLK_FPGA1, U32 XC95288XL-TQ144, U33 XCF02S, U35 74LS245, U36 74LS245, U37 74LS245, U4 PAC_GHOST, U42 74LS245, U43 74LVC245, U44 74LS245, U46 74LS541, U47 74LS541, U48 74LS541, U49 74LS541, U50 74LS245, U51 74LS245, U52 74LS245, U53 74LVC245, U54 74LS245, U55 74LS245, U6 POWER_SELECT, U7 74LS14, U9 LDO_REG_7805

Commit message: Z80-FPGA-SBC: schematic edits
Source: Z80 Board ANTS_MOD 2/ECB SBC V2 (working folder): SBC.sch, SBC-cache.lib.
Parts:
- added P3: CLK_SEL, ~, symbol CONN_3X2
Connections:
- wire segments 1455 -> 1469
- no-connect marks 87 -> 86
Changed lines of the file:
@@
 LIBS:Z8S180
 LIBS:z53c80
-LIBS:ANTS_MOD1
-LIBS:74xgxx
-LIBS:ac-dc
 LIBS:adc-dac
 LIBS:analog_switches
@@
 LIBS:contrib
 LIBS:cypress
-LIBS:dc-dc
 LIBS:device
 LIBS:digital-audio
 LIBS:display
 LIBS:dsp
-LIBS:elec-unifil
-LIBS:ftdi
 LIBS:gennum
 LIBS:graphic
 LIBS:interface
 LIBS:linear
-LIBS:logo
-LIBS:microchip_pic10mcu
-LIBS:microchip_pic12mcu
-LIBS:microchip_pic16mcu
 LIBS:microcontrollers
-LIBS:msp430
-LIBS:nxp_armmcu
 LIBS:opto
 LIBS:philips
 LIBS:power
-LIBS:powerint
 LIBS:pspice
-LIBS:references
 LIBS:regul
-LIBS:relays
-LIBS:sensors
 LIBS:siliconi
-LIBS:stm8
-LIBS:stm32
-LIBS:supertex
 LIBS:SymbolsSimilarEN60617+oldDIN617
 LIBS:texas
@@
 LIBS:video
 LIBS:xxx
+LIBS:ANTS_MOD1
 LIBS:SBC-cache
 EELAYER 27 0
@@
 Sheet 1 1
 Title ""
-Date "25 aug 2013"
+Date "12 sep 2013"
 Rev ""
 Comp ""
@@
 	17850 7850 17300 7850
 Wire Wire Line
-	2350 3400 1800 3400
-Wire Wire Line
 	3850 1900 3350 1900
 Wire Wire Line
@@
 Wire Wire Line
 	16350 3700 15750 3700
-Connection ~ 1800 3400
 Wire Wire Line
 	5750 6600 5750 6300
@@
 	22700 22250 23300 22250
 Wire Wire Line
-	24650 22650 25250 22650
+	22700 22650 23300 22650
 Wire Wire Line
 	22700 22750 23300 22750
@@
 NoConn ~ 17000 18050
 NoConn ~ 17000 17950
-NoConn ~ 23300 23150
 NoConn ~ 23300 22950
 NoConn ~ 23300 22850
@@
 Text Label 22750 22550 0    60   ~ 0
 sXTRQ*
-Text Label 24700 22650 0    60   ~ 0
+Text Label 22750 22650 0    60   ~ 0
 A19
 Text Label 22750 22750 0    60   ~ 0
@@
 Text Label 1250 8000 0    60   ~ 0
 /CS_UART
-Text Label 1900 3400 0    60   ~ 0
+Text Label 2900 4350 0    60   ~ 0
 CLK_CPU
 Text Label 3400 3700 0    60   ~ 0
@@
 Wire Wire Line
 	4900 14800 5650 14800
-Wire Wire Line
-	3850 14700 4500 14700
-Wire Wire Line
-	4500 15800 3850 15800
 Text Label 4500 16300 0    60   ~ 0
 -16V
@@
 +16V
 Wire Wire Line
-	4400 16000 4500 16000
-Wire Wire Line
-	4400 16000 4400 16300
-Wire Wire Line
 	4400 16300 4500 16300
 Wire Wire Line
-	4500 14900 4400 14900
-Wire Wire Line
-	4400 14900 4400 15200
+	4400 14700 4400 15200
 Wire Wire Line
 	4400 15200 4500 15200
@@
 PHI_CLOCK
 Wire Wire Line
-	22400 22650 23300 22650
-Text Label 22400 22650 0    60   ~ 0
+	22400 23150 23300 23150
+Text Label 22400 23150 0    60   ~ 0
 CLOCK2
 Text Label 17150 29600 0    60   ~ 0
@@
 Text Notes 32450 29250 1    60   ~ 0
 to FPGA
-Text Label 31700 31100 2    60   ~ 0
+Text Label 1450 4550 2    60   ~ 0
 PHI_CLOCK
-Text Label 31700 31000 2    60   ~ 0
+Text Label 1450 4450 2    60   ~ 0
 CLK_CPU2
 Wire Wire Line
@@
 Text Notes 32850 20900 1    60   ~ 0
 to LED's
+Wire Wire Line
+	4400 14700 4500 14700
+Wire Wire Line
+	3850 14700 4300 14700
+Wire Wire Line
+	4300 14700 4300 14900
+Wire Wire Line
+	4300 14900 4500 14900
+Wire Wire Line
+	3850 15800 4300 15800
+Wire Wire Line
+	4300 15800 4300 16000
+Wire Wire Line
+	4300 16000 4500 16000
+Wire Wire Line
+	4500 15800 4400 15800
+Wire Wire Line
+	4400 15800 4400 16300
+$Comp
+L CONN_3X2 P3
+U 1 1 5223CF89
+P 2300 4500
+F 0 "P3" H 2300 4750 50  0000 C CNN
+F 1 "CLK_SEL" V 2300 4550 40  0000 C CNN
+F 2 "~" H 2300 4500 60  0000 C CNN
+F 3 "~" H 2300 4500 60  0000 C CNN
+	1    2300 4500
+	1    0    0    -1
+$EndComp
+Wire Wire Line
+	2900 4350 2700 4350
+Wire Wire Line
+	2700 4550 2800 4550
+Wire Wire Line
+	2800 4550 2800 4350
+Connection ~ 2800 4350
+Wire Wire Line
+	2700 4450 2800 4450
+Connection ~ 2800 4450
+Wire Wire Line
+	1800 3400 1950 3400
+Wire Wire Line
+	1950 3400 1950 4050
+Wire Wire Line
+	1950 4050 1650 4050
+Wire Wire Line
+	1650 4050 1650 4350
+Wire Wire Line
+	1650 4350 1900 4350
+Wire Wire Line
+	1900 4450 1450 4450
+Wire Wire Line
+	1450 4550 1900 4550
 $EndSCHEMATC
