File: Backplane-18-Slot/rev1/S100-Backplane.sch (KiCad schematic (older format))
At the start: 185 parts, among them IC1 7805, IC2 LM4250, J4000 USB_2, J9002 ISP_M2, K1 RESET(s), K4000 I/O V?, P1 CONN_4, P10 CONN_1, P11 CONN_1, P12 CONN_2, P13 CONN_1, P14 CONN_1, P15 CONN_1, P16 CONN_1, P17 CONN_1, P18 CONN_1, P19 S100_MALE, P20 XILINX CABLE, P21 CLK_CPU, P25 CLK_SEL, P3 CONN_1, P4 CONN_1, P4000 FT232R I/O, P6 CONN_1, P7 CONN_1, P8 CONN_1, P9 CONN_1, P9000 ATX_POWER_24, P9001 ATX_POWER, P9002 POWER_SW, P9003 CONN_1, P9004 CONN_1, P9005 CONN_1, P9006 CONN_1, Q1 2N3906, Q13 2N3904, Q2 2N3904, Q3 TIP29, Q4 TIP30, Q5 ^^NPN-BC817-SOT323, Q9001 2N3904, Q9002 2N3904, SW1 SW_PUSH, SW2 PROG_B, SW9000 POWER, U1 S100, U10 S100, U100 S100-EX, U1000 ^^LOGO1, U1001 LOGO2, U11 S100, U12 S100, U13 S100, U14 S100, U15 S100, U16 S100, U17 S100, U18 74LS541, U2 S100, U20 74LVC245, U21 74LVC245, U22 74LVC245, U23 74LS14, U24 74LVC245, U25 74HC245, U27 74LVC245, U3 S100, U30 XC6SLX9-TQ144, U31 23LC1024, U32 XCF02S, U33 CLK_FPGA1, U34 LDO_REG_7805, U35 LM1086CS, U36 LF25CDT, U37 LD1117DT12, U4 S100, U4000 FT232R, U45 74LVC245, U5 S100, U6 S100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

Commit message: Backplane-18-Slot rev1: remove FPGA/USB section; PIC18F1330 PSU; trimpot, D44C/D45C; new gerbers
Source: S100 Backplane ANTS_MOD/S100 Backplane-001/BACKUPS/backup 18102013 1134/S100 Backplane-001
Parts:
- removed C10, C11, C14, C15, C17, C19, C22, C23, C25, C26, C27: 0.1 uF, symbol C
- removed C28, C29, C30, C31, C32, C33, C34, C35: 10 uF, symbol CP
- removed D2, D3, D4, D5, D6: LED, symbol LED
- removed D4000: TX, symbol LED
- removed D4001: RX, symbol LED
- removed J4000: USB_2, symbol USB_2
- removed J9002: ISP_M2, symbol RJ12
- removed JP10, JP4, JP5, JP6, JP7, JP8, JP9: JUMPER, PIN_ARRAY_2X1, symbol JUMPER
- removed K4000: I/O V?, ~, symbol CONN_3
- removed P19: S100_MALE, S100_MALE, symbol S100_MALE
- removed P20: XILINX CABLE, symbol CONN_5X2
- removed P21: CLK_CPU, symbol DIL14
- removed P25: CLK_SEL, ~, symbol CONN_3X2
- removed P4000: FT232R I/O, symbol CONN_10
- removed Q3: TIP29, TO220, symbol TIP29
- removed Q4: TIP30, TO220, symbol TIP30
- removed Q5: ^^NPN-BC817-SOT323, symbol ^^NPN-BC817-SOT323
- removed R18, R19, R20, R24, R25, R26, R29, R4000, R4001: 330, symbol R
- removed R21, R22, R23: 100, symbol R
- removed R27: 10K, symbol R
- removed R28, R30: 4K7, symbol R
- removed R31: 1K, symbol R
- removed SW2: PROG_B, symbol SW_PUSH
- removed U18: 74LS541, symbol 74LS541
- removed U20, U21, U22, U24, U27, U45: 74LVC245, ~, symbol 74LVC245
- removed U23: 74LS14, symbol 74LS14
- removed U25: 74HC245, symbol 74HC245
- removed U30: XC6SLX9-TQ144, symbol XC6SLX9-TQ144
- removed U31: 23LC1024, symbol 23LC1024
- removed U32: XCF02S, symbol XCF02S
- removed U33: CLK_FPGA1, symbol CRYSTAL_OSC_SMD
- removed U34: LDO_REG_7805, ~, symbol LDO_REG_7805
- removed U35: LM1086CS, symbol LM1086CS
- removed U36: LF25CDT, symbol LF25CDT
- removed U37: LD1117DT12, symbol LD1117DT12
- removed U4000: FT232R, symbol FT232R
- removed U9000: PIC18F2550, symbol PIC18F2550
- added C9005: 0.47 UF, symbol CP
- added P9007: PIC_ISP, symbol CONN_6
- added Q3: TIP29-D44C, transistor-TO220, symbol -NPN-TO220
- added Q4: TIP30/D45C, transistor-TO220, symbol -PNP-TO220
- added U23: 74LS04, ~, symbol 74LS04
- added U9000: PIC18F1330, symbol PIC18F1330
- P1: value CONN_4 -> POWER BLOCK
- P9002: value POWER_SW -> EX_POWER_BUTTON
- R1: value 2000 -> TRIMPOT
Connections:
- net labels removed: +16V, +16Vi, +8Vi, -16V, -16Vi, -GND, 0V, 0V_Ai, 0V_Bi, 0V_Ci, 0Vi, 25LC_CS, 25LC_S0, 25LC_SCK, 25LC_SI, A0bi, A0y, A10bi, A10y, A11bi, A11y, A12bi, A12y, A13bi, A13y, A14bi, A14y, A15bi, A15y, A16bi, A16y, A17bi, A17y, A18bi, A18y, A19bi, A19y, A1bi, A1y, A20, A20bi, A20y, A21, A21bi, A21y, A22bi, A22y, A23bi, A23y, A2bi, A2y, A3bi, A3y, A4bi, A4y, A5bi, A5y, A6bi, A6y, A7bi, A7y, A8bi, A8y, A9bi, A9y, ADSB*i, CDSB*i, CLK_TIMER, CLOCK*i, CTS_TTL, D0, D1, D2, D3, D4, D5, D6, D7, DBUSIN_EN, DBUSOUT_EN, DI0bi, DI1bi, DI2bi, DI3bi, DI4bi, DI5bi, DI6bi, DI7bi, DO0bi, DO1bi, DO2bi, DO3bi, DO4bi, DO5bi, DO6bi, DO7bi, DODSB*i, DSR_TTL, DTR_TTL, ERROR*i, FPGA_10, FPGA_100, FPGA_101, FPGA_102, FPGA_104, FPGA_105, FPGA_11, FPGA_111, FPGA_112, FPGA_114, FPGA_115, FPGA_116, FPGA_117, FPGA_118, FPGA_119, FPGA_12, FPGA_120, FPGA_121, FPGA_123, FPGA_124, FPGA_126, FPGA_127, FPGA_131, FPGA_132, FPGA_133, FPGA_134, FPGA_137, FPGA_138, FPGA_139, FPGA_14, FPGA_140, FPGA_141, FPGA_142, FPGA_15, FPGA_16, FPGA_17, FPGA_2, FPGA_21, FPGA_22, FPGA_23, FPGA_24, FPGA_26, FPGA_27, FPGA_29, FPGA_30, FPGA_32, FPGA_33, FPGA_34, FPGA_35, FPGA_45, FPGA_46, FPGA_48, FPGA_5, FPGA_55, FPGA_56, FPGA_57, FPGA_58, FPGA_59, FPGA_6, FPGA_7, FPGA_78, FPGA_79, FPGA_8, FPGA_80, FPGA_81, FPGA_82, FPGA_83, FPGA_84, FPGA_87, FPGA_88, FPGA_9, FPGA_92, FPGA_93, FPGA_94, FPGA_95, FPGA_97, FPGA_98, FPGA_99, FPGA_CLK_0, FPGA_CLK_2, FT_VCCIO, HOLD*i, INT*i, IOREQbi, MAIN_VCC, MWRTi, NDEF1i, NDEF2i, NDEF3i, NMI*i, PF1_TDI, PF1_TDO, PHANTOM*i, PHI_CLOCK, PHIi, POC*i, PWRFAIL*i, RDYi, RESET*i, RFU1i, RFU2i, RFU3, RFU4i, RTS_TTL, RX, S6LX9_TD0, S6LX9_TDI, SDSB*i, SIN_TTL, SIXTN*i, SLAVE_CLR*i, SOUT_TTL, TCK, TMA0*i, TMA1*i, TMA2*i, TMA3*i, TMS, TX, USB_VCC0, V1.2, V2.5, V3.3, VI0*i, VI1*i, VI2*i, VI3*i, VI4*i, VI5*i, VI6*i, VI7*i, XRDYi, pDBINi, pHLDAi, pSTVAL*i, pSYNCi, pWR*i, sHLTAi, sINPi, sINTAi, sM1i, sMEMRi, sOUTi, sWO*i, sXTRQ*i
- wire segments 2878 -> 2137
- no-connect marks 67 -> 3
Other:
- note added: "LOW when PSU is OFF\nHIGH when PSU is ON"
- note added: "NPN TO-220\n1=B\n2=C\n3=E\n4=C"
- note added: "PNP TO-220\n1=B\n2=C\n3=E\n4=C"
- note added: "Pin 54 on S100 Connector"
- note added: "Pin 75 on S100 Connector"
- note added: "Reset Circuit"
- note removed: "+3.3V from Power supply on Rail"
- note removed: "+5V from Power supply on Rail"
- note removed: "/WAIT is output from slave to Processor"
- note removed: "2CCLK"
- note removed: "ADDRESS INPUTS from S100 BUS"
- note removed: "All routed to CPLD"
- note removed: "B -> A"
- note removed: "BANK 0"
- note removed: "BANK 1"
- note removed: "BANK 2"
- note removed: "BANK 3"
- note removed: "CONFIG"
- note removed: "DATA I/O from/to S100 BUS"
- note removed: "DATA RD/WR"
- note removed: "DIN"
- note removed: "DONE_LED"
- note removed: "DPAK"
- note removed: "INIT_B"
- note removed: "INPUT"
- note removed: "INPUT from S100 BUS"
- note removed: "INPUTS to FPGA"
- note removed: "Input in terms of the Slave on the S100\nBus, DI is INPUT for salve, so, OUTPUT\nfor master"
- note removed: "Jumper to exclude Program Flash 1 from Chain\njump 2->4, for inclusion jump 1->2 & 3->4"
- note removed: "Jumper to exclude S3E 1 from Chain\njump 2->4, for inclusion jump 1->2 & 3->4"
- note removed: "MASTER input"
- note removed: "MODE Selector"
- note removed: "OUTPUT"
- note removed: "OUTPUT from Slave on S100 Bus,\nINPUT for the Master"
- note removed: "OUTPUT to S100 BUS"
- note removed: "PROG_B"
- note removed: "Pin 1 => FT232R Transmit Asynchronous Data Output.\nPin 5 => FT232R Receiving Asynchronous Data Input."
- note removed: "Pin 15 (Address line 18) S100 Bus"
- note removed: "Pin 16 (Address line 16) S100 Bus"
- note removed: "Pin 17 (Address line 17) S100 Bus"
- note removed: "Pin 24 (Primary Processor clock line ) Input"
- note removed: "Pin 44 (processor Instruction Fetch Cycle M1) Input"
- note removed: "Pin 45 (I/O WR) Input"
- note removed: "Pin 46 (I/O RD) Input"
- note removed: "Pin 47 (MEM RD) Input"
- note removed: "Pin 49 (clock line from another board) Input"
- note removed: "Pin 5 (RXD) - INPUT\nPin 1 (TXD) - OUTPUT"
- note removed: "Pin 54 (reset from another board) Input"
- note removed: "Pin 59 (Address line 19) S100 Bus"
- note removed: "Pin 61 (Address line 20) S100 Bus"
- note removed: "Pin 62 (Address line 21) S100 Bus"
- note removed: "Pin 63 (I/O REQUEST) Input"
- note removed: "Pin 65 (MEM REQUEST) Input"
- note removed: "Pin 68 (MEM WR) Input"
- note removed: "Pin 72 (controld run/WAIT state of processor) Input"
- note removed: "Pin 75 (forces processor to reset state) Input"
- note removed: "Pin 77 (active low when processor write to I/O or MEM) Input"
- note removed: "Pin 78 (active high when processor reads I/O or MEM) Input"
- note removed: "Pin 79 (Address line 0) S100 Bus"
- note removed: "Pin 97 (active low when processor is in Write status) Input"
- note removed: "RX"
- note removed: "TO-220"
- note removed: "TTL SERIAL to USB BREAKOUT"
- note removed: "TX"
- note removed: "XILINX CABLE HEADER\n1, 3, 5, 7, 9, 11, 13 - GND\n2 - VREF +3.3V\n4 - TMS\n6 - TCK\n8 - TDO\n10 - TDI\n12, 14 - NC"
- note removed: "from Pin 13 of CPLD"
- note removed: "from Pin 18 of CPLD"
- note removed: "~IORQ"
- note removed: "~MREQ"
- note removed: "~RD"
- note removed: "~WR"
- moved on the sheet: C1, C13, C2, C3, C4, C5, C6, C7, C8, C9002, C9003, D1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

Commit message: Backplane-18-Slot rev1: add P25-P28 bus headers; reset RC 10R/10uF
Source: S100 Backplane ANTS_MOD/S100 Backplane-001/BACKUPS/backup 19102013 1942/S100 Backplane-001
Parts:
- removed C13: 0.1 uF, symbol C
- added C13: 10uF, symbol CP
- added C9: 0.1 uF, symbol C
- added P19, P2, P20, P21, P22, P23, P24, P5: CONN_1, symbol CONN_1
- added P25, P26, P27, P28: CONN_13X2, symbol CONN_13X2
- R15: value 1K -> 10
Connections:
- wire segments 2137 -> 2245
Other:
- note added: "POWER CONNECTOR"
- note added: "POWER ON LED"
- moved on the sheet: C1, C2, C3, C4, C5, C6, C7, C8, D1, D12, IC1, IC2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
