File: Backplane-18-Slot/rev1/S100-Backplane.sch (KiCad schematic (older format))
At the start: 124 parts, among them IC1 7805, IC2 LM4250, K1 RESET(s), P1 POWER BLOCK, P10 CONN_1, P11 CONN_1, P12 CONN_2, P13 CONN_1, P14 CONN_1, P15 CONN_1, P16 CONN_1, P17 CONN_1, P18 CONN_1, P19 CONN_1, P2 CONN_1, P20 CONN_1, P21 CONN_1, P22 CONN_1, P23 CONN_1, P24 CONN_1, P25 CONN_13X2, P26 CONN_13X2, P27 CONN_13X2, P28 CONN_13X2, P3 CONN_1, P4 CONN_1, P5 CONN_1, P6 CONN_1, P7 CONN_1, P8 CONN_1, P9 CONN_1, P9000 ATX_POWER_24, P9001 ATX_POWER, P9002 EX_POWER_BUTTON, P9003 CONN_1, P9004 CONN_1, P9005 CONN_1, P9006 CONN_1, P9007 PIC_ISP, Q1 2N3906, Q13 2N3904, Q2 2N3904, Q3 TIP29-D44C, Q4 TIP30/D45C, Q9001 2N3904, Q9002 2N3904, SW1 SW_PUSH, SW9000 POWER, U1 S100, U10 S100, U100 S100-EX, U1000 ^^LOGO1, U1001 LOGO2, U11 S100, U12 S100, U13 S100, U14 S100, U15 S100, U16 S100, U17 S100, U2 S100, U23 74LS04, U3 S100, U4 S100, U5 S100, U6 S100, U7 S100, U8 S100, U9 S100, U9000 PIC18F1330

Commit message: Backplane-18-Slot rev1: Rev 1.0 final: ATX PSU split off, 15.7x8.0 in board, gerbers and BOM
Source: S100 Backplane ANTS_MOD/S100 Backplane-001/S100 Backplane-001
S100-Backplane.pro is taken from S100 Backplane ANTS_MOD/V1 - backup 22-10-2015 (same content, saved 2013-10-20); the working-folder copy was only re-saved in 2016.
Parts:
- removed C9002, C9003: 0.1 uF, symbol C
- removed C9005: 0.47 UF, symbol CP
- removed D9002, D9003: LED, symbol LED
- removed P9000: ATX_POWER_24, ~, symbol ATX_POWER_24
- removed P9001: ATX_POWER, symbol CONN_5
- removed P9002: EX_POWER_BUTTON, symbol CONN_2
- removed P9003, P9004, P9005, P9006: CONN_1, symbol CONN_1
- removed P9007: PIC_ISP, symbol CONN_6
- removed Q9001, Q9002: 2N3904, symbol NPN
- removed R9000, R9002: 330, symbol R
- removed R9001, R9009: 470, symbol R
- removed R9004, R9008: 10k, symbol R
- removed SW9000: POWER, symbol SW_PUSH
- removed U9000: PIC18F1330, symbol PIC18F1330
Connections:
- net labels removed: +3.3V_B, +5V_B, -12V_B, 12V, 5VSB, ATX_PWRUP, ATX_PWR_OK, GND_B, M2_MCLR, M2_PGC, M2_PGD, M2_VDD, ~PS_ON
- wire segments 2245 -> 2134
- no-connect marks 3 -> 2
Other:
- note removed: "ATX 24 Pin Supply Control Circuit & Plug"
- note removed: "LOW when PSU is OFF\nHIGH when PSU is ON"
