File: S6LX9-FPGA-IO/TMRINT.sch (KiCad schematic (older format))
At the start: 97 parts, among them P1 CLK TIMER 2, P19 S100_MALE, P2 I/O, P20 XILINX CABLE, P21 CLK TIMER 1, P25 CLK_SEL, P6 CONN_1, P7 CONN_1, Q5 ^^NPN-BC817-SOT323, SW2 PROG_B, U1 LTC3419, U18 74LS541, U2 74LVC245, U20 74LVC245, U21 74LVC245, U22 74LVC245, U24 74LVC245, U27 74LVC245, U3 74HC245, U30 XC6SLX9-TQ144, U31 23LC1024, U32 XCF02S, U33 CLK_FPGA1, U34 LDO_REG_7805, U35 LM1086CS_TO252_DPAK, U4 DS1302, U45 74LVC245, U5 7432, U6 74LVC245, U7 74LVC245, X1 32.768KHz

Commit message: S6LX9-FPGA-IO: schematic tweaks (R1 4K8 to 6K8), placement
Source: S100 FPGA_TIMER_INT_CONTROLLER/backups/03112013 0658 (KiCad project TMRINT, original folder name FPGA_TIMER_INT_CONTROLLER)
Parts:
- R1: value 4K8 -> 6K8
Connections:
- net labels added: 3.3b, POT CLK 1, POT CLK 2
- wire segments 956 -> 957
Other:
- note added: "R2 should equal 6750 ohm for 3.3V output\nwith 1K5 ohm for R1"
- note removed: "R2 should equal 4750 ohm for 2.5V output\nwith 1K5 ohm for R1"
Changed lines of the file:
@@
 	23300 8900 24400 8900
 Wire Wire Line
-	24250 14650 25350 14650
-Wire Wire Line
-	24250 14450 25350 14450
-Wire Wire Line
-	24250 14250 25350 14250
-Wire Wire Line
-	24250 14050 25350 14050
-Wire Wire Line
-	24250 13750 25350 13750
-Wire Wire Line
-	24250 13550 25350 13550
-Wire Wire Line
-	24250 13350 25350 13350
-Wire Wire Line
-	24250 13150 25350 13150
-Wire Wire Line
 	27400 22950 28100 22950
 Wire Wire Line
@@
 Connection ~ 6400 10050
 Wire Wire Line
-	24250 13050 25350 13050
-Wire Wire Line
-	24250 13250 25350 13250
-Wire Wire Line
-	24250 13450 25350 13450
-Wire Wire Line
-	24250 13650 25350 13650
-Wire Wire Line
 	18600 12450 18400 12450
 Wire Wire Line
@@
 	18400 13450 18600 13450
 Wire Wire Line
-	24250 13950 25350 13950
-Wire Wire Line
-	24250 14150 25350 14150
-Wire Wire Line
-	24250 14350 25350 14350
-Wire Wire Line
-	24250 14550 25350 14550
-Wire Wire Line
 	23300 8800 24400 8800
 Wire Wire Line
@@
 Text Label 18600 14150 0    60   ~ 0
 FPGA_118
-Text Label 24250 13950 0    60   ~ 0
+Text Label 25100 14650 2    60   ~ 0
 FPGA_132
-Text Label 24250 14050 0    60   ~ 0
+Text Label 25100 14550 2    60   ~ 0
 FPGA_131
-Text Label 24250 14150 0    60   ~ 0
+Text Label 25100 14450 2    60   ~ 0
 FPGA_127
-Text Label 24250 14250 0    60   ~ 0
+Text Label 25100 14350 2    60   ~ 0
 FPGA_126
-Text Label 24250 14350 0    60   ~ 0
+Text Label 25100 14250 2    60   ~ 0
 FPGA_124
-Text Label 24250 14450 0    60   ~ 0
+Text Label 25100 14150 2    60   ~ 0
 FPGA_123
-Text Label 24250 14550 0    60   ~ 0
+Text Label 25100 14050 2    60   ~ 0
 FPGA_121
-Text Label 24250 14650 0    60   ~ 0
+Text Label 25100 13950 2    60   ~ 0
 FPGA_120
 Text Label 18600 14050 0    60   ~ 0
@@
 Text Label 18600 13250 0    60   ~ 0
 FPGA_132
-Text Label 24250 13750 0    60   ~ 0
+Text Label 25100 13050 2    60   ~ 0
 FPGA_133
-Text Label 24250 13650 0    60   ~ 0
+Text Label 25100 13150 2    60   ~ 0
 FPGA_134
-Text Label 24250 13550 0    60   ~ 0
+Text Label 25100 13250 2    60   ~ 0
 FPGA_137
-Text Label 24250 13450 0    60   ~ 0
+Text Label 25100 13350 2    60   ~ 0
 FPGA_138
-Text Label 24250 13350 0    60   ~ 0
+Text Label 25100 13450 2    60   ~ 0
 FPGA_139
-Text Label 24250 13250 0    60   ~ 0
+Text Label 25100 13550 2    60   ~ 0
 FPGA_140
-Text Label 24250 13150 0    60   ~ 0
+Text Label 25100 13650 2    60   ~ 0
 FPGA_141
-Text Label 24250 13050 0    60   ~ 0
+Text Label 25100 13750 2    60   ~ 0
 FPGA_142
 Text Label 10650 12600 0    60   ~ 0
@@
 P 8400 3550
 F 0 "R1" V 8480 3550 50  0000 C CNN
-F 1 "4K8" V 8400 3550 50  0000 C CNN
+F 1 "6K8" V 8400 3550 50  0000 C CNN
 F 2 "" H 8400 3550 60  0001 C CNN
 F 3 "" H 8400 3550 60  0001 C CNN
@@
 CLOCKS & OSCILLATORS
 Text Label 7350 2650 0    60   ~ 0
-V2.5
+3.3b
 Text Notes 8300 3700 0    59   ~ 0
 "R2"
@@
 Vout = 0.6*( 1+ (R2/R1) )\n\nR2 = R1*( (Vout/0.6) -  1)
 Text Notes 7100 3850 0    39   ~ 0
-R2 should equal 4750 ohm for 2.5V output\nwith 1K5 ohm for R1
+R2 should equal 6750 ohm for 3.3V output\nwith 1K5 ohm for R1
 Text Label 36900 31050 0    60   ~ 0
 VI0*i
@@
 	40850 3100 41000 3100
 Wire Wire Line
-	41850 3750 41150 3750
+	41150 3750 42000 3750
 Wire Wire Line
 	41150 3750 41150 4850
@@
 	1    0    0    -1
 $EndComp
-Text Label 30550 29950 0    60   ~ 0
-V5.0
 Text Label 30550 30750 0    60   ~ 0
 GND
@@
 	19550 3850 19550 3950
 Connection ~ 19800 3950
+Text Label 30550 29950 0    60   ~ 0
+3.3b
+Text Label 42000 3750 0    60   ~ 0
+POT CLK 2
+Text Label 40200 4150 2    60   ~ 0
+POT CLK 1
+Wire Wire Line
+	40200 4150 40450 4150
+Connection ~ 40450 4150
+Connection ~ 41850 3750
+Wire Wire Line
+	25350 13050 25100 13050
+Wire Wire Line
+	25100 13150 25350 13150
+Wire Wire Line
+	25350 13250 25100 13250
+Wire Wire Line
+	25100 13350 25350 13350
+Wire Wire Line
+	25100 13450 25350 13450
+Wire Wire Line
+	25350 13550 25100 13550
+Wire Wire Line
+	25100 13650 25350 13650
+Wire Wire Line
+	25350 13750 25100 13750
+Wire Wire Line
+	25100 13950 25350 13950
+Wire Wire Line
+	25350 14050 25100 14050
+Wire Wire Line
+	25350 14150 25100 14150
+Wire Wire Line
+	25100 14250 25350 14250
+Wire Wire Line
+	25350 14350 25100 14350
+Wire Wire Line
+	25100 14450 25350 14450
+Wire Wire Line
+	25350 14550 25100 14550
+Wire Wire Line
+	25100 14650 25350 14650
 $EndSCHEMATC

Commit message: S6LX9-FPGA-IO: add six FPGA LEDs and FPGA I/O header P3
Source: S100 FPGA_TIMER_INT_CONTROLLER/backups/03112013 1002 (KiCad project TMRINT, original folder name FPGA_TIMER_INT_CONTROLLER)
Parts:
- added D1, D7, D8: LED, symbol LED
- added P3: FPGA I/O, symbol CONN_10
- added R7, R8, R9: 330, symbol R
Connections:
- net labels added: FPGA_1, FPGA_144, FPGA_66, FPGA_67, FPGA_74, FPGA_75
- wire segments 957 -> 987
- no-connect marks 52 -> 46
Other:
- note added: "to LED's"
- moved on the sheet: C21, JP10

Commit message: S6LX9-FPGA-IO: add data buffer U8, U18 74LS541 to 74HC245; first routed PCB
Source: S100 FPGA_TIMER_INT_CONTROLLER/backups/17112013 1254 (KiCad project TMRINT, original folder name FPGA_TIMER_INT_CONTROLLER)
Parts:
- removed C10: 0.1 uF, symbol C
- removed U18: 74LS541, symbol 74LS541
- added Cx? (x2): 10 uF, symbol CP
- added U18: 74HC245, symbol 74HC245
- added U8: 74LVC245, ~, symbol 74LVC245
- added Ux?: ^^3.3VREG_SOT223, ~, symbol ^^3.3VREG_SOT223
Connections:
- net labels added: V3.3b
- net labels removed: 0V
- wire segments 987 -> 1007
Other:
- note added: "AMS1117 1.2V Reg (same as 3.3v fixed version)"
- note added: "SOT233"
- moved on the sheet: JP4, JP5, JP6, JP7, JP8, JP9, P3

Commit message: S6LX9-FPGA-IO: 1.2 V LDO replaces LTC3419, add M25P80, final routing, gerbers and BOM
Source: S100 FPGA_TIMER_INT_CONTROLLER (working folder). TMRINT.sch and TMRINT-cache.lib carry a 2015-08-04 re-save mtime; TMRINT.sch is byte-identical to TMRINT.bak (2014-06-23) and its part list matches TMRINT.net (2014-03-11), so the commit is dated from the PCB, netlist, gerbers and BOM.
Parts:
- removed C1, C5: 22uF, symbol C
- removed C2, C4: 22pF, symbol C
- removed C3: 10uF, symbol C
- removed JP10: JUMPER, PIN_ARRAY_2X1, symbol JUMPER
- removed L1, L2: 3.3uH, ~, symbol INDUCTOR
- removed U1: LTC3419, symbol LTC3419
- added U9: M25P80, ~, symbol M25P80
- R1: value 6K8 -> 3K3; Digikey (none) -> ??
- R2, R3, R4: value 1K5 -> 10K; Digikey (none) -> ??
- gave numbers to parts that had none: 3
Connections:
- net labels added: M25P_CS
- wire segments 1007 -> 986
- no-connect marks 46 -> 45
Other:
- note added: "Part Number\nRS# 663-0240\nor\nRS# 540-8134 (preferance)\n"
- note removed: ""R1""
- note removed: ""R2""
- note removed: "MSOP 10 0.5mm"
- note removed: "Part Number\nRS# 663-2870"
