File: Flash-UART/S100_B1FU.kicad_pcb (KiCad board)
At the start: 2 copper layers, 254 x 134.1 mm, 161 parts, among them P1 M25P80 ISP, P19 XILINX CABLE2, P3 CONN_2, P4 S100_MALE, P5 PIC_ISP, P6 CONN_1, P7 CONN_1, P8 CONN_2, P9 CONN_2, Q1 ^^NPN-SOT23, Q2 ^^NPN-SOT23, Q3 ^^NPN-SOT23, Q4 ^^NPN-SOT23, Q5 ^^NPN-SOT23, Q6 ^^NPN-SOT23, Q7 ^^NPN-SOT23, Q8 ^^NPN-SOT23, Q9 ^^NPN-SOT23, SW1 RESET, SW2 RESET, SW4 FLASH_SELECT, SW50 FLASH/RUN, U1 LDO_REG_7805, U11 ^^74LS541, U12 ^^74LV244, U14 M25P80, U15 M25P80, U16 M25P80, U17 M25P80, U18 CH341A, U19 ^^74LS541, U2 LM1086CS, U20 XC95288XL-TQ144, U3din1 ^^74LS541, U3dout1 ^^74LS541, U4 ^^74LS541, U5 ^^74LS541, U6 ^^74LS541, U7a1 74HC245, U7b1 74HC245, U8 PIC18F1330, X1 12MHz

Commit message: Flash-UART: routed PCB and gerbers; add CPLD I/O headers P2/P10
Source: S100_B1FLASHUART/backups/05052014 FINAL after printed
Gerbers dated 2014-04-16; one GND label added to the schematic on 2014-04-18.
The working folder S100_B1FLASHUART/ is identical apart from a KiCad autosave.
Parts:
- added C3: 0.1 uF, C2, F.Cu at (85.8, 152.8)
- added P10: CONN_4, SIL-4, F.Cu at (174.7, 120.5)
- added P2: CONN_4, SIL-4, F.Cu at (174.6, 129.3)
Connections:
- C19 pad 1: /V3.3_CLPD_IO -> /V3.3
- C26 pad 1: /V3.3_CLPD_INT -> /V3.3
- C33 pad 1: /V3.3_CLPD_INT -> /V3.3
- C34 pad 1: /V3.3_CLPD_IO -> /V3.3
- C35 pad 1: /V3.3_CLPD_IO -> /V3.3
- C36 pad 1: /V3.3_CLPD_IO -> /V3.3
- C37 pad 1: /V3.3_CLPD_IO -> /V3.3
- C38 pad 1: /V3.3_CLPD_IO -> /V3.3
- C39 pad 1: /V3.3_CLPD_IO -> /V3.3
- C40 pad 1: /V3.3_CLPD_IO -> /V3.3
- P8 pad 1: /V3.3_CLPD_INT -> /V3.3
- P9 pad 1: /V3.3_CLPD_IO -> /V3.3
- R20 pad 2: (no net) -> /BOARD_SEL_LED
- R7 pad 2: (no net) -> /DONE_LED
- U18 pad 27: (no net) -> GND
- U20 pad 1: /V3.3_CLPD_IO -> /V3.3
- U20 pad 109: /V3.3_CLPD_IO -> /V3.3
- U20 pad 110: (no net) -> N-0000071
- U20 pad 111: (no net) -> N-0000074
- U20 pad 112: (no net) -> N-0000076
- U20 pad 113: (no net) -> N-0000093
- U20 pad 115: (no net) -> N-0000095
- U20 pad 116: (no net) -> N-0000097
- U20 pad 127: /V3.3_CLPD_IO -> /V3.3
- U20 pad 141: /V3.3_CLPD_INT -> /V3.3
- U20 pad 30: (no net) -> /DONE_LED
- U20 pad 31: (no net) -> /BOARD_SEL_LED
- U20 pad 33: (no net) -> /SLAVE_CLR*vv
- U20 pad 37: /V3.3_CLPD_IO -> /V3.3
- U20 pad 42: /V3.3_CLPD_INT -> /V3.3
- U20 pad 55: /V3.3_CLPD_IO -> /V3.3
- U20 pad 73: /V3.3_CLPD_IO -> /V3.3
- U20 pad 8: /V3.3_CLPD_INT -> /V3.3
- U20 pad 84: /V3.3_CLPD_INT -> /V3.3
- U7a1 pad 9: (no net) -> /SLAVE_CLR*vv
Routing:
- net GND: track 0.00 -> 1951.3 mm, vias 0 -> 62
- net VCC: track 0.00 -> 809.3 mm
- net /V3.3: track 0.00 -> 679.1 mm, vias 0 -> 15
- net /D1: track 0.00 -> 268.5 mm, vias 0 -> 7
- net /D0: track 0.00 -> 252.0 mm, vias 0 -> 6
- net /D3: track 0.00 -> 233.7 mm, vias 0 -> 4
- net /D2: track 0.00 -> 231.2 mm, vias 0 -> 4
- net /IOREQbb: track 0.00 -> 228.5 mm, vias 0 -> 3
- net /D7: track 0.00 -> 227.4 mm, vias 0 -> 4
- net /D4: track 0.00 -> 226.5 mm, vias 0 -> 4
- net /D6: track 0.00 -> 223.9 mm, vias 0 -> 4
- net /D5: track 0.00 -> 205.5 mm, vias 0 -> 2
- net /SLAVE_CLR*: track 0.00 -> 198.0 mm, vias 0 -> 3
- net /BOARD_INTERRUPT_VECTc: track 0.00 -> 187.8 mm, vias 0 -> 6
- net /Q2: track 0.00 -> 181.9 mm, vias 0 -> 4
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- added copper zone on B.Cu, net GND
- added copper zone on F.Cu, net GND
Other:
- net class Dafault big clearance: trace_width 0.254 -> 0.25
- board text added: "B_S"
- board text added: "D2"
- board text added: "D3"
- board text added: "F0 F1 F2 F3"
- board text added: "FLASH ICP"
- board text added: "F_SEL"
- board text added: "GND CLK Din CS Dout"
- board text added: "GND P110 P111 P112"
- board text added: "GND P116 P115 P113"
- board text added: "RDY (P72)"
- board text added: "RESET (P75)"
- board text added: "RS232 / TMA / FLASH LOADER © 2014 Antony Burrows ALL RIGHTS RESERVED"
- board text added: "RS232 | TMA | Serial Flash Board Rev 1.0"
- board text added: "TMA0 TMA1 TMA2 TMA3"
- board text added: "U11"
- board text added: "U19"
- board text added: "U20"
- board text added: "U3Din"
- board text added: "U3Dout"
- board text added: "U4"
- board text added: "U5"
- board text added: "U6"
- board text added: "U8"
- board text added: "XC95288XL-TQ144"
- board text removed: "UART / TMA /EPROM LOADER © 2014 Antony Burrows ALL RIGHTS RESERVED"
