File: Flash-UART/S100_B1FU.sch (KiCad schematic (older format))
At the start: 161 parts, among them P1 M25P80 ISP, P19 XILINX CABLE2, P3 CONN_2, P4 S100_MALE, P5 PIC_ISP, P6 CONN_1, P7 CONN_1, P8 CONN_2, P9 CONN_2, Q1 ^^NPN-SOT23, Q2 ^^NPN-SOT23, Q3 ^^NPN-SOT23, Q4 ^^NPN-SOT23, Q5 ^^NPN-SOT23, Q6 ^^NPN-SOT23, Q7 ^^NPN-SOT23, Q8 ^^NPN-SOT23, Q9 ^^NPN-SOT23, SW1 RESET, SW2 RESET, SW4 FLASH_SELECT, SW50 FLASH/RUN, U1 LDO_REG_7805, U11 ^^74LS541, U12 ^^74LV244, U14 M25P80, U15 M25P80, U16 M25P80, U17 M25P80, U18 CH341A, U19 ^^74LS541, U2 LM1086CS, U20 XC95288XL-TQ144, U3din1 ^^74LS541, U3dout1 ^^74LS541, U4 ^^74LS541, U5 ^^74LS541, U6 ^^74LS541, U7a1 74HC245, U7b1 74HC245, U8 PIC18F1330, X1 12MHz

Commit message: Flash-UART: routed PCB and gerbers; add CPLD I/O headers P2/P10
Source: S100_B1FLASHUART/backups/05052014 FINAL after printed
Gerbers dated 2014-04-16; one GND label added to the schematic on 2014-04-18.
The working folder S100_B1FLASHUART/ is identical apart from a KiCad autosave.
Parts:
- added C3: 0.1 uF, symbol C
- added P10, P2: CONN_4, symbol CONN_4
Connections:
- net labels removed: CPLD_1, ~BOARD_SELECT
- wire segments 1101 -> 1129
Other:
- note removed: "to U7c output buffer to S100 Bus - RESET*"
Changed lines of the file:
@@
 Sheet 1 1
 Title "noname.sch"
-Date "14 apr 2014"
+Date "16 apr 2014"
 Rev ""
 Comp ""
@@
 Text Label -7100 23850 0    60   ~ 0
 GND
-Text Label 32600 22600 2    60   ~ 0
-CPLD_1
 Text Label -7250 29450 2    60   ~ 0
 RESETtoS100
-Text Notes 30150 22600 0    60   ~ 0
-to U7c output buffer to S100 Bus - RESET*
 Text Notes 50150 23150 0    87   ~ 0
 SPARE CPLD PINS
@@
 Text Label 40500 8900 2    60   ~ 0
 DONE_LED
-Text Label 32600 22900 2    60   ~ 0
-~BOARD_SELECT
 Wire Notes Line
 	39250 7000 45700 7000
@@
 Wire Wire Line
 	29850 19000 30150 19000
+$Comp
+L C C3
+U 1 1 534BCA00
+P 3500 6500
+F 0 "C3" H 3550 6600 50  0000 L CNN
+F 1 "0.1 uF" H 3550 6400 50  0000 L CNN
+F 2 "" H 3500 6500 60  0001 C CNN
+F 3 "" H 3500 6500 60  0001 C CNN
+	1    3500 6500
+	1    0    0    -1
+$EndComp
+Wire Wire Line
+	32600 22700 32950 22700
+Wire Wire Line
+	32950 22800 32600 22800
+Wire Wire Line
+	32950 23000 32600 23000
+$Comp
+L CONN_4 P2
+U 1 1 534DBECF
+P 42000 24300
+F 0 "P2" V 41950 24300 50  0000 C CNN
+F 1 "CONN_4" V 42050 24300 50  0000 C CNN
+F 2 "" H 42000 24300 60  0000 C CNN
+F 3 "" H 42000 24300 60  0000 C CNN
+	1    42000 24300
+	1    0    0    -1
+$EndComp
+$Comp
+L CONN_4 P10
+U 1 1 534DBEDC
+P 42000 24750
+F 0 "P10" V 41950 24750 50  0000 C CNN
+F 1 "CONN_4" V 42050 24750 50  0000 C CNN
+F 2 "" H 42000 24750 60  0000 C CNN
+F 3 "" H 42000 24750 60  0000 C CNN
+	1    42000 24750
+	1    0    0    -1
+$EndComp
+Wire Wire Line
+	39150 24600 40200 24600
+Wire Wire Line
+	40200 24600 40200 24900
+Wire Wire Line
+	40200 24900 41650 24900
+Wire Wire Line
+	39150 24500 40250 24500
+Wire Wire Line
+	40250 24500 40250 24800
+Wire Wire Line
+	40250 24800 41650 24800
+Wire Wire Line
+	39150 24400 40300 24400
+Wire Wire Line
+	40300 24400 40300 24700
+Wire Wire Line
+	40300 24700 41650 24700
+Wire Wire Line
+	39150 24300 40500 24300
+Wire Wire Line
+	40500 24300 40500 24450
+Wire Wire Line
+	40500 24450 41650 24450
+Wire Wire Line
+	39150 24200 40550 24200
+Wire Wire Line
+	40550 24200 40550 24350
+Wire Wire Line
+	40550 24350 41650 24350
+Wire Wire Line
+	39150 24100 40650 24100
+Wire Wire Line
+	40650 24100 40650 24250
+Wire Wire Line
+	40650 24250 41650 24250
+Text Label 41650 24000 0    60   ~ 0
+GND
+Wire Wire Line
+	41650 24000 41400 24000
+Wire Wire Line
+	41400 24000 41400 24600
+Wire Wire Line
+	41400 24600 41650 24600
+Wire Wire Line
+	41650 24150 41400 24150
+Connection ~ 41400 24150
+Text Label 42850 21700 0    60   ~ 0
+V3.3
+Text Label 42850 21800 0    60   ~ 0
+V3.3
+Text Label 42550 21700 2    60   ~ 0
+V3.3_CLPD_IO
+Text Label 42550 21800 2    60   ~ 0
+V3.3_CLPD_INT
+Wire Wire Line
+	42850 21700 42550 21700
+Wire Wire Line
+	42550 21800 42850 21800
+Text Label 19450 11400 0    60   ~ 0
+GND
+Wire Wire Line
+	19450 11400 19100 11400
 $EndSCHEMATC
