File: Z80-CPU/v3/s100_Z80 V3.kicad_pcb (KiCad board)
At the start: 2 copper layers, 254 x 134.6 mm, 166 parts, among them K1 CONN_3, K10 U15 Clock, K2 CONN_3, K3 pSYNCdata, K4 CONN_3, K5 pSYNC, K6 U35p12, K7 U40p8, K8 WRstrobe, K9 U29B Q, P1 S100_MALE, P2 CONN_4X2, P3 CLK_CPU, P34 CONN_1, P35 CONN_1, P36 CONN_3X2, P4 CONN_2X2, P5 CLK_CPU, P6 MASTER_OSC, P7 CLK_SEL, Q1 2N3904, Q2 ^^NPN-SOT23, Q3 ^^NPN-SOT23, Q4 ^^NPN-SOT23, Q5 ^^NPN-SOT23, Q6 ^^NPN-SOT23, Q7 ^^NPN-SOT23, SW1 DIPS_08, SW2 DIPS_08, SW3 DIPS_08, SW4 DIPS_08, U1 Z80, U10 74LS165, U11 74LS165, U12 ^^74LS541, U13 2732, U14 74LS682N, U15 74LS165, U16 74LS273, U17 74LS273, U18 74LS161, U19 ^^74LS541, U2 ^^74LS541, U20 ^^74LS541, U21 ^^74LS541, U22 ^^74LS541, U23 74LS02, U24 74LS04, U25 74LS04, U26 74LS05, U27 74LS139, U28 74LS00, U29 74LS74, U3 ^^74LS541, U31 74LS00, U33 74LS74, U34 74LS74, U35 74LS32, U36 74LS04, U37 74LS05, U38 74F04, U39 74S08, U4 74LS153, U40 74S00, U43 74LS11, U44 74LS32, U45 74LS02, U47 74LS04, U48 LDO_REG_7805, U49 74LS00, U5 74LS157, U6 74LS153, U7 74LS32, U8 74LS157, U9 74LS165

Commit message: Z80-CPU v3: schematic and placement rework
Source: S100 Z80 version3/backups/17-07-2014 0138
Parts:
- removed C42: 22 uF, C1V7
- removed C43: 33 uF, C1V7
- removed C48, C63, C7: 0.1 uF, C2
- removed D6: 1N4148, D3
- removed JP4, JP5, JP6, JP7: JUMPER, SIL-2
- removed Q1: 2N3904, TO92-INVERT
- removed R11: 4700, R3
- removed RR8, RR9: 1000, r_pack9
- removed U26: 74LS05, DIP-14__300_ELL
- removed U44: 74LS32, DIP-14__300_ELL
- removed U49: 74LS00, DIP-14__300_ELL
- added K11: bA13, SIL-3, F.Cu at (75.2, 120.6)
- added K12: bA12, SIL-3, F.Cu at (78.2, 120.6)
- added K13: bA19, SIL-3, F.Cu at (57.7, 120.6)
- added K14: bA18, SIL-3, F.Cu at (60.6, 120.6)
- added K15: bA16, SIL-3, F.Cu at (66.5, 120.6)
- added K16: bA17, SIL-3, F.Cu at (63.6, 120.6)
- K6: value U35p12 -> bA15
- K7: value U40p8 -> bA14
- U39: value 74S08 -> 74LS02
- moved K7 188.2 mm to (72.3, 120.6)
- moved U24 92.5 mm to (171.4, 90.2)
- moved U36 78.8 mm to (171.4, 62.2)
- moved K3 77.8 mm to (185.0, 62.4)
- moved K6 76.5 mm to (69.4, 120.6)
- moved C2 76.4 mm to (121.9, 90.2)
- moved R5 64.2 mm to (248.9, 54.6), turned to 180 degrees
- moved P6 40.8 mm to (237.6, 33.0), turned to 0 degrees
- moved U27 33.5 mm to (99.1, 90.2)
- moved U31 33.3 mm to (97.8, 34.3)
- moved U29 29.7 mm to (64.5, 34.3)
- moved P7 28.0 mm to (247.0, 33.0), turned to 0 degrees
- moved K10 17.9 mm to (22.6, 88.9)
- moved SW1 15.4 mm to (37.1, 90.2)
- moved U12 15.2 mm to (67.8, 105.4)
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Connections:
- K10 pad 3: /MEM_WAIT -> /CLK_CPU
- K3 pad 3: N-00000111 -> N-00000142
- K5 pad 1: (no net) -> N-0000077
- K6 pad 1: N-00000154 (its old number) -> /bA15
- K6 pad 2: N-00000155 (its old number) -> N-0000093
- K6 pad 3: GND -> N-0000094
- K7 pad 1: N-00000147 (its old number) -> /bA14
- K7 pad 2: /sWO* -> N-0000095
- K7 pad 3: N-00000148 (its old number) -> N-0000096
- P1 pad 10: /PU1K-HH -> (no net)
- P1 pad 11: /PU1K-II -> (no net)
- P1 pad 14: /PU1K-U -> (no net)
- P1 pad 4: /PU1K-BB -> (no net)
- P1 pad 5: /PU1K-CC -> (no net)
- P1 pad 54: /PU1K-I -> (no net)
- P1 pad 55: /PU1K-X -> (no net)
- P1 pad 56: /PU1K-W -> (no net)
- P1 pad 57: /PU1K-V -> (no net)
- P1 pad 6: /PU1K-DD -> (no net)
- P1 pad 67: /PHANTOM* -> (no net)
- P1 pad 7: /PU1K-EE -> (no net)
- P1 pad 75: /PU1K-P -> /RESET*
- P1 pad 8: /PU1K-FF -> (no net)
- P1 pad 9: /PU1K-GG -> (no net)
- P1 pad 99: /POC* -> (no net)
- P36 pad 3: /MEM_WAIT -> /MREQ+
- P7 pad 2: /CLK -> /CLK_CPU
- P7 pad 4: /CLK -> /CLK_CPU
- P7 pad 6: /CLK -> /CLK_CPU
- P7 pad 8: /CLK -> /CLK_CPU
- R5 pad 2: /CLK -> /CLK_CPU
- RR5 pad 10: /PU1K-I -> (no net)
- RR5 pad 2: (no net) -> /PU1K-JJ
- RR6 pad 10: (no net) -> /ERROR*
- RR6 pad 4: (no net) -> /NMI*
- RR6 pad 5: /NMI* -> /PU1K-N
- RR6 pad 6: /PU1K-N -> (no net)
- RR6 pad 7: /POC* -> /CDSB*
- RR6 pad 8: /PU1K-P -> /PU1K-T
- RR6 pad 9: /PU1K-Q -> /PU1K-Y
- RR7 pad 10: /PU5K-G -> (no net)
- RR7 pad 4: (no net) -> /PU5K-C
- RR7 pad 8: /PU5K-G -> (no net)
- U1 pad 26: /PU1K-P -> /RESET*
- U1 pad 6: /CLK -> /CLK_CPU
- U10 pad 2: /CLK -> /CLK_CPU
- U11 pad 2: /CLK -> /CLK_CPU
- U12 pad 1: /ADSB -> GND
- U12 pad 19: GND -> /ADSB
- U15 pad 7: (no net) -> N-0000077
- U16 pad 1: N-0000029 (its old number) -> /PU5K-C
- U17 pad 1: N-0000029 (its old number) -> /PU5K-C
- U21 pad 2: /READ_STROBE -> /RD+
- U21 pad 4: N-00000111 -> N-00000142
- U21 pad 5: N-00000148 (its old number) -> /pWR*b
- U21 pad 8: N-0000019 (its old number) -> /MWRTb
- U22 pad 11: (no net) -> /PU5K-C
- U22 pad 3: N-00000328 -> /sOUTb
- U22 pad 4: N-0000036 (its old number) -> N-00000100
- U22 pad 5: /MEM_RD -> /sMEMRb
- U22 pad 6: /sWO* -> /WR*
- U22 pad 8: N-0000021 -> /sINTAb
- U22 pad 9: (no net) -> /RESET*
- U24 pad 4: N-00000148 (its old number) -> /pWR*b
- U25 pad 13: /REFSH* -> (no net)
- U28 pad 12: /sOUT -> /sOUTb
- U28 pad 9: /READ_STROBE -> /RD+
- U3 pad 2: N-0000044 -> N-0000093
- U3 pad 3: N-000003 (its old number) -> N-0000095
- U3 pad 4: N-0000043 -> N-0000097
- U3 pad 5: N-000004 -> N-0000026
- U31 pad 10: /IORQ -> /IORQ+
- U33 pad 11: /CLK -> /CLK_CPU
- U34 pad 10: /PU1K-P -> /RESET*
- U35 pad 1: /PU1K-P -> N-0000034
- U35 pad 11: /READ_STROBE -> (no net)
- U35 pad 12: N-00000155 (its old number) -> (no net)
- U35 pad 13: /RD+ -> (no net)
- U35 pad 2: /PU1K-P -> N-0000037
- U35 pad 3: N-0000029 (its old number) -> N-000004
- U36 pad 10: N-00000153 (its old number) -> N-00000142
- U36 pad 11: N-00000154 (its old number) -> N-00000179
- U36 pad 12: N-0000021 -> /PU1K-J
- U36 pad 13: N-0000035 (its old number) -> /BUSAK*
- U36 pad 3: /CLK -> /CLK_CPU
- U38 pad 10: /MEM_WAIT -> /MREQ+
- U38 pad 6: /IORQ -> /IORQ+
- U39 pad 1: /WR+ -> /sOUTb
- U39 pad 10: /MEM_WAIT -> /sMEMRb
- U39 pad 11: N-0000036 (its old number) -> /sOUTb
- U39 pad 12: /IORQ -> /pWR*b
- U39 pad 13: /RD+ -> /MWRTb
- U39 pad 2: /IORQ -> /WR*
- U39 pad 3: N-00000328 -> /IORQ*
- U39 pad 4: N-00000160 (its old number) -> N-00000100
- U39 pad 5: /IORQ* -> /RD*
- U39 pad 6: N-00000111 -> /IORQ*
- U39 pad 8: /MEM_RD -> /RD*
- U39 pad 9: /RD+ -> /MREQ*
- U4 pad 7: N-000004 -> N-0000099
- U4 pad 9: N-0000043 -> N-0000098
- U40 pad 10: /RD* -> /sMEMRb
- U40 pad 12: N-00000160 (its old number) -> N-00000112
- U40 pad 2: /MEM_WAIT -> /MREQ+
- U40 pad 3: N-00000160 (its old number) -> N-00000112
- U40 pad 4: /M1+ -> N-00000112
- U40 pad 5: /IORQ -> /IORQ*
- U40 pad 6: N-0000035 (its old number) -> N-00000179
- U40 pad 8: N-00000147 (its old number) -> /27_ROM_OE
- U40 pad 9: N-00000153 (its old number) -> N-00000218
- U45 pad 10: N-00000154 (its old number) -> /sINTAb
- U45 pad 4: N-0000019 (its old number) -> (no net)
- U45 pad 5: N-00000148 (its old number) -> (no net)
- U45 pad 6: N-00000328 -> (no net)
- U47 pad 1: N-00000143 (its old number) -> N-000004
- U47 pad 2: N-00000311 -> N-00000218
- U5 pad 12: /bA16 -> N-0000085
- U5 pad 4: /bA19 -> N-0000087
- U5 pad 7: /bA18 -> N-0000088
- U5 pad 9: /bA17 -> N-0000089
- U6 pad 7: N-000003 (its old number) -> N-0000096
- U6 pad 9: N-0000044 -> N-0000094
- U7 pad 11: N-00000137 (its old number) -> N-0000037
- U7 pad 8: N-00000134 -> N-0000034
- U9 pad 2: /CLK -> /CLK_CPU
Routing:
- added copper zone on F.Cu, net GND
Other:
- net class Default: trace_width 0.23 -> 0.24
- board text added: "pSYNC"

Commit message: Z80-CPU v3: schematic and placement
Source: S100 Z80 version3/backups/17-07-2014 1631
Parts:
- added D9: D2-1, ^^LED-0805, F.Cu at (82.3, 82.0)
- added K17: EN_WAITS, SIL-3, F.Cu at (152.5, 97.7)
- added R42: 330, ^^SMD_Resistor-0805, B.Cu at (77.2, 82.0)
- D8: value POWER -> D2-1
- moved K3 46.5 mm to (222.2, 90.3)
- moved R35 34.3 mm to (222.4, 120.8)
- moved R36 34.3 mm to (224.9, 120.8)
- moved R2 33.3 mm to (46.9, 31.1)
- moved Q2 33.3 mm to (45.5, 35.3)
- moved R1 33.3 mm to (44.3, 31.1)
- moved Q3 9.40 mm to (37.8, 35.2)
- moved R3 9.40 mm to (39.4, 31.1)
- moved R6 9.40 mm to (36.8, 31.1)
- moved K4 5.40 mm to (114.9, 67.2)
- moved R38 2.92 mm to (230.0, 120.8)
- moved R37 2.92 mm to (227.5, 120.8)
- moved K9 2.05 mm to (191.8, 82.3)
- moved K2 2.05 mm to (185.4, 82.3)
- moved K5 2.05 mm to (188.6, 82.3)
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Connections:
- RR7 pad 10: (no net) -> /PU1K-waits
- RR7 pad 8: (no net) -> /PU1K-cp1
- RR7 pad 9: (no net) -> /PU1K-cp2
- U16 pad 11: N-0000054 (its old number) -> /PU1K-cp1
- U17 pad 11: N-000007 -> /PU1K-cp2
- U17 pad 16: (no net) -> N-000005
- U24 pad 12: N-000009 (its old number) -> N-00000107
- U27 pad 6: N-0000054 (its old number) -> /PU1K-cp1
- U27 pad 7: N-000007 -> /PU1K-cp2
- U43 pad 1: N-000009 (its old number) -> N-00000104

Commit message: Z80-CPU v3: routed REV 2.0 board and gerbers
Source: S100 Z80 version3/backups/20-07-2014
Newest file is 2014-07-18 00:18 (the gerber time); the folder name says 20-07.
Parts:
- added U26: ^^LOGO1, ***Z80cpuV32, F.Cu at (230.3, 143.3)
Routing:
- net GND: track 0.00 -> 2096.9 mm, vias 0 -> 73
- net VCC: track 0.00 -> 1274.5 mm, vias 0 -> 1
- net /D1: track 0.00 -> 372.3 mm, vias 0 -> 4
- net N-00000316: track 0.00 -> 371.6 mm, vias 0 -> 3
- net /D7: track 0.00 -> 365.4 mm, vias 0 -> 2
- net /bA6: track 0.00 -> 365.2 mm, vias 0 -> 4
- net /D2: track 0.00 -> 357.7 mm, vias 0 -> 4
- net /D0: track 0.00 -> 347.8 mm, vias 0 -> 4
- net /bA4: track 0.00 -> 346.1 mm, vias 0 -> 4
- net /D6: track 0.00 -> 339.2 mm, vias 0 -> 2
- net /bA7: track 0.00 -> 334.6 mm, vias 0 -> 4
- net /bA5: track 0.00 -> 334.0 mm
- net /D3: track 0.00 -> 328.4 mm, vias 0 -> 2
- net /D5: track 0.00 -> 327.6 mm, vias 0 -> 5
- net /bA3: track 0.00 -> 325.8 mm, vias 0 -> 2
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- added copper zone on B.Cu, net GND
Other:
- outline, holes or cut-outs redrawn
- board text removed: "Z80 CPU BOARD"

Commit message: Z80-CPU v3: schematic changes after the gerbers (unrouted board)
Source: S100 Z80 version3/backups/20-07-2014 1447
Parts:
- removed U43: 74LS11, DIP-14__300_ELL
- removed U47: 74LS04, DIP-14__300_ELL
- added C5: 0.1 uF, C2, F.Cu at (85.1, 34.3)
- added K18: ROM_E-, SIL-3, F.Cu at (24.6, 47.0)
- added R11: 10K, R3, F.Cu at (114.0, 47.0)
- added R16: 10K, R3, F.Cu at (116.6, 47.0)
- added U30: ^^74LS541, DIP-20__300_ELL, F.Cu at (138.4, 34.3)
- added U32: ^^74LS541, DIP-20__300_ELL, F.Cu at (138.4, 47.2)
- added U41: ^^74LS541, DIP-20__300_ELL, F.Cu at (101.6, 34.3)
- moved U29 91.5 mm to (34.3, 120.7)
- moved C58 91.4 mm to (21.8, 120.7)
- moved K4 87.1 mm to (30.2, 47.0)
- moved U13 76.5 mm to (59.4, 40.6)
- moved C59 73.7 mm to (51.8, 120.7)
- moved U31 65.2 mm to (64.3, 90.2)
- moved U35 63.2 mm to (97.8, 47.0)
- moved C49 63.2 mm to (85.1, 47.0)
- moved C15 36.8 mm to (121.9, 34.3)
- moved C53 36.8 mm to (121.9, 47.0)
- moved RR5 34.5 mm to (100.5, 128.3)
- moved R4 25.7 mm to (47.5, 132.3), turned to 270 degrees
- moved D1 25.4 mm to (53.3, 25.9)
- moved D8 20.4 mm to (48.0, 129.0)
- moved C6 17.6 mm to (52.1, 134.1)
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Connections:
- K17 pad 2: N-00000104 -> N-0000079
- P6 pad 2: N-0000032 -> N-000005
- P6 pad 4: N-0000032 -> N-000005
- RR2 pad 10: (no net) -> /RR4p10
- RR4 pad 10: /RR4p10 -> (no net)
- U13 pad 1: /bA7 -> N-00000100
- U13 pad 10: /D1 -> N-00000126
- U13 pad 11: /D2 -> N-00000127
- U13 pad 13: /D3 -> N-00000128
- U13 pad 14: /D4 -> N-00000129
- U13 pad 15: /D5 -> N-00000130
- U13 pad 16: /D6 -> N-00000131
- U13 pad 17: /D7 -> N-00000124
- U13 pad 18: GND -> N-00000135
- U13 pad 19: /bA10 -> N-00000123
- U13 pad 2: /bA6 -> N-00000101
- U13 pad 20: /27_ROM_OE -> N-00000115
- U13 pad 21: /bA11 -> N-00000120
- U13 pad 22: /bA9 -> N-00000121
- U13 pad 23: /bA8 -> N-00000122
- U13 pad 3: /bA5 -> N-00000102
- U13 pad 4: /bA4 -> N-00000103
- U13 pad 5: /bA3 -> N-00000104
- U13 pad 6: /bA2 -> N-00000105
- U13 pad 7: /bA1 -> N-00000106
- U13 pad 8: /bA0 -> N-00000107
- U13 pad 9: /D0 -> N-00000125
- U17 pad 19: N-000002 (its old number) -> /ROM_E-
- U18 pad 1: VCC -> (no net)
- U18 pad 2: N-0000032 -> (no net)
- U24 pad 5: (no net) -> N-00000111
- U24 pad 6: (no net) -> N-00000112
- U25 pad 12: (no net) -> /WAIT*
- U25 pad 13: (no net) -> N-00000113
- U28 pad 4: (no net) -> /PU1K-D
- U28 pad 5: (no net) -> /PU1K-E
- U28 pad 6: (no net) -> N-00000111
- U31 pad 1: (no net) -> N-0000079
- U31 pad 2: (no net) -> N-00000112
- U31 pad 3: (no net) -> N-00000113
- U35 pad 3: N-0000039 (its old number) -> N-0000027
- U36 pad 1: (no net) -> N-0000027
- U36 pad 2: (no net) -> N-00000215
- U36 pad 5: (no net) -> /27_ROM_OE
- U36 pad 6: (no net) -> /ROM_SELECT
- U40 pad 9: N-00000220 -> N-00000215
- U7 pad 9: N-000002 (its old number) -> /ROM_E-
Routing:
- net GND: track 2096.9 -> 0.00 mm, vias 73 -> 0
- net VCC: track 1274.5 -> 0.00 mm, vias 1 -> 0
- net /D1: track 372.3 -> 0.00 mm, vias 4 -> 0
- net N-00000351: track 371.6 -> 0.00 mm, vias 3 -> 0
- net /D7: track 365.4 -> 0.00 mm, vias 2 -> 0
- net /bA6: track 365.2 -> 0.00 mm, vias 4 -> 0
- net /D2: track 357.7 -> 0.00 mm, vias 4 -> 0
- net /D0: track 347.8 -> 0.00 mm, vias 4 -> 0
- net /bA4: track 346.1 -> 0.00 mm, vias 4 -> 0
- net /D6: track 339.2 -> 0.00 mm, vias 2 -> 0
- net /bA7: track 334.6 -> 0.00 mm, vias 4 -> 0
- net /bA5: track 334.0 -> 0.00 mm
- net /D3: track 328.4 -> 0.00 mm, vias 2 -> 0
- net /D5: track 327.6 -> 0.00 mm, vias 5 -> 0
- net /bA3: track 325.8 -> 0.00 mm, vias 2 -> 0
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- added copper zone on B.Cu, net (none)
- added copper zone on F.Cu, net (none)
- removed copper zone on B.Cu, net GND
- removed copper zone on F.Cu, net GND
