File: Z80-CPU/v3/s100_Z80 V3.kicad_pcb (KiCad board)
At the start: 2 copper layers, 254 x 134.6 mm, 140 parts, among them K1 CONN_3, K10 U15 Clock, K11 bA13, K12 bA12, K13 bA19, K14 bA18, K15 bA16, K16 bA17, K17 EN_WAITS, K18 ROM_E-, K2 CONN_3, K3 pSYNCdata, K4 CONN_3, K5 pSYNC, K6 bA15, K7 bA14, K8 WRstrobe, K9 U29B Q, P1 S100_MALE, P2 CONN_4X2, P3 CLK_CPU, P34 CONN_1, P35 CONN_1, P36 CONN_3X2, P4 CONN_2X2, P5 CLK_CPU, P6 MASTER_OSC, P7 CLK_SEL, P8 CONN_20, P9 CONN_20, Q1 NPN, Q2 NPN, Q3 NPN, SW1 DIPS_08, SW2 DIPS_08, SW3 DIPS_08, SW4 DIPS_08, U1 Z80, U10 74LS165, U11 74LS165, U12 ^^74LS541, U13 2732, U14 74LS682N, U15 74LS165, U18 74LS161, U19 ^^74LS541, U2 ^^74LS541, U20 ^^74LS541, U21 ^^74LS541, U22 ^^74LS541, U24 74LS04, U25 74LS04, U26 ^^LOGO1, U27 74LS139, U28 74LS00, U29 74LS74, U3 ^^74LS541, U30 ^^74LS541, U31 74LS00, U32 ^^74LS541, U33 74LS74, U34 74LS74, U35 74LS32, U36 74LS04, U37 74LS05, U38 74F04, U39 74LS02, U40 74S00, U41 ^^74LS541, U45 74LS02, U48 LDO_REG_7805, U7 74LS32, U8 74LS157, U9 74LS165

Commit message: Z80-CPU v3: final schematic and routed board
Source: S100 Z80 version3/backups/S100 Z80 version3 (a full copy of the v3 working folder as of 2014-08-09; its nested backups are the same as the ones already committed).
The gerbers are still the 2014-07-18 set, made before the July 20-26 changes.
Parts:
- U32: value ^^74LS541 -> 74HCT541
Connections:
- P6 pad 2: N-0000032 (its old number) -> N-0000034
- P6 pad 4: N-0000032 (its old number) -> N-0000034
- U18 pad 1: (no net) -> VCC
- U18 pad 2: (no net) -> N-0000034
Routing:
- net GND: track 0.00 -> 1614.2 mm, vias 0 -> 8
- net VCC: track 0.00 -> 1074.4 mm
- net /bA2: track 0.00 -> 411.3 mm, vias 0 -> 3
- net /bA3: track 0.00 -> 367.2 mm, vias 0 -> 3
- net /bA5: track 0.00 -> 367.0 mm, vias 0 -> 4
- net /CLK_CPU: track 0.00 -> 356.0 mm, vias 0 -> 5
- net /PU5K-C: track 0.00 -> 353.2 mm, vias 0 -> 3
- net /bA6: track 0.00 -> 346.4 mm, vias 0 -> 4
- net /D7: track 0.00 -> 340.5 mm, vias 0 -> 3
- net /bA4: track 0.00 -> 334.0 mm, vias 0 -> 1
- net /D5: track 0.00 -> 333.0 mm, vias 0 -> 3
- net /bA7: track 0.00 -> 329.0 mm, vias 0 -> 5
- net /sWO*b: track 0.00 -> 321.2 mm, vias 0 -> 1
- net /D4: track 0.00 -> 317.5 mm, vias 0 -> 1
- net /D1: track 0.00 -> 310.2 mm, vias 0 -> 5
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