File: SRAM-8MB/rev2/s100_SRAMp2.sch (KiCad schematic (older format))
At the start: 147 parts, among them IC2 74LS682N, IC3 74LS682N, P1 S100_MALE, P10 CONN_10, P11 CONN_6, P2 CONN_8, P3 CONN_8, P34 CONN_1, P35 CONN_1, P4 CONN_8, P5 CONN_8, P6 CONN_8, P7 CONN_8, P8 CONN_10, P9 XILINX CABLE2, Q1 ^^NPN-BC817-SOT323, Q10 ^^NPN-BC817-SOT323, Q11 ^^NPN-BC817-SOT323, Q12 ^^NPN-BC817-SOT323, Q13 ^^NPN-BC817-SOT323, Q14 ^^NPN-BC817-SOT323, Q15 ^^NPN-BC817-SOT323, Q16 ^^NPN-BC817-SOT323, Q2 ^^NPN-BC817-SOT323, Q3 ^^NPN-BC817-SOT323, Q4 ^^NPN-BC817-SOT323, Q5 ^^NPN-BC817-SOT323, Q6 ^^NPN-BC817-SOT323, Q7 ^^NPN-BC817-SOT323, Q9 ^^NPN-BC817-SOT323, SW2 DIPS_08, SW3 DIPS_08, SW4 DIPS_08, U1 LDO_REG_7805, U19 74LS245, U2 ^^74LS541, U21 SRAM_512KB, U22 74LS245, U23 ^^74LS541, U24 ^^74LS541, U26 SRAM_512KB, U27 74LS165, U29 SRAM_512KB, U31 ^^74LS541, U32 SRAM_512KB, U33 SRAM_512KB, U34 SRAM_512KB, U35 SRAM_512KB, U36 SRAM_512KB, U37 SRAM_512KB, U38 SRAM_512KB, U39 SRAM_512KB, U4 XC9572XL-TQ100, U40 SRAM_512KB, U41 SRAM_512KB, U42 SRAM_512KB, U43 SRAM_512KB, U44 SRAM_512KB, U45 LOGO_S100_SRAM_8MB, U5 74LS06, U6 ^^74LS541, U7 ^^74LS541

Commit message: SRAM-8MB rev2: schematic re-saved (WAIT-disable jumper JP4, block tidy)
Source: S100 8MB SRAM Proto2/ (working folder schematic, 2015-07-17)
Parts:
- added JP4: JUMPER, PIN_ARRAY_2X1, symbol JUMPER
Connections:
- wire segments 1184 -> 1189
Other:
- moved on the sheet: C11, C12, C14, C15, C16, C17, C18, C2, C20, C21, C22, C25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
