File: Z80-CPU/v2/s100_Z80 V2.sch (KiCad schematic (older format))
At the start: 163 parts, among them K1 CONN_3, K2 CONN_3, K4 CONN_3, P1 S100_MALE, P2 CONN_4X2, P3 CLK_CPU, P34 CONN_1, P35 CONN_1, P36 CONN_3X2, P37 CONN_2X2, P4 CONN_2X2, P5 CLK_CPU, P6 CLK_SEL, Q1 2N3904, Q2 ^^NPN-SOT23, Q3 ^^NPN-SOT23, Q4 ^^NPN-SOT23, Q5 ^^NPN-SOT23, Q6 ^^NPN-SOT23, Q7 ^^NPN-SOT23, SW2 DIPS_08, SW3 DIPS_08, SW4 DIPS_08, U1 Z80, U10 74LS165, U11 74LS165, U12 74LS373, U13 2732, U14 74LS682N, U16 74LS273, U17 74LS273, U19 74LS244, U2 74LS373, U20 74LS244, U21 74LS244, U22 74LS373, U23 74LS02, U24 74LS04, U25 74LS04, U26 74LS05, U27 74LS139, U28 74LS00, U29 74LS74, U3 74LS373, U30 74LS74, U31 74LS00, U32 74LS74, U33 74LS74, U34 74LS74, U35 74LS32, U36 74LS04, U37 74LS05, U38 74F04, U39 74S08, U4 74LS153, U40 74S00, U41 74LS27, U42 2.0000 MHz, U43 74LS11, U44 74LS32, U45 74LS02, U47 74LS04, U48 LDO_REG_7805, U49 74LS00, U5 74LS157, U6 74LS153, U7 74LS32, U8 74LS157, U9 74LS165

Commit message: Z80-CPU v2: schematic notes and rework wiring (WR+/RD+)
Source: S100 Z80 version2/s100_Z80 V2.sch and -cache.lib (working folder).
Connections:
- wire segments 1209 -> 1214
Other:
- note added: "A14"
- note added: "A15"
- note added: "RD+"
- note added: "WR+"
- note added: "b0"
- note added: "b1"
- note added: "b2"
- note added: "b3"
- note added: "b4"
- note added: "b5"
- note added: "b6"
- note added: "b7"
- note added: "port 0 Q4 - bit3"
- note added: "port 0 Q5 - bit2"
- note added: "port 1 Q4 - bit3"
- note added: "port 1 Q5 - bit2"
- note added: "port D2"
- note added: "port D3"
Changed lines of the file:
@@
 Sheet 1 1
 Title "noname.sch"
-Date "6 jun 2014"
+Date "10 aug 2015"
 Rev ""
 Comp ""
@@
 	5500 21300 5500 21700
 Wire Wire Line
-	10200 20850 10200 21550
-Wire Wire Line
 	3250 21550 3250 18500
 Wire Wire Line
@@
 Connection ~ 15950 22150
 Wire Wire Line
-	10200 21550 15950 21550
+	10200 21550 17850 21550
 Connection ~ 18950 31050
 Connection ~ 19200 25950
@@
 	20850 20450 20850 22700
 Wire Wire Line
-	19800 23900 17850 23900
-Wire Wire Line
-	17850 23900 17850 22150
+	17850 23900 19800 23900
 Wire Wire Line
-	17850 22150 17250 22150
+	17850 21550 17850 23900
 Connection ~ 11400 24000
 Wire Wire Line
@@
 	17650 17450 17650 24300
 Connection ~ 8050 24100
-Wire Wire Line
-	7600 24100 8450 24100
 Connection ~ 4800 23900
 Wire Wire Line
@@
 	18150 6950 19300 6950
 Wire Wire Line
-	19300 6950 19300 8250
-Wire Wire Line
 	19300 8250 18400 8250
 Connection ~ 18150 6750
@@
 	3100 25150 8450 25150
 Wire Wire Line
-	8450 25150 8450 24300
+	8450 25150 8450 24100
 Connection ~ 11400 22450
 Wire Wire Line
@@
 Connection ~ 17950 20350
 Wire Wire Line
-	15950 21550 15950 22900
-Wire Wire Line
 	2850 20300 2850 21800
 Connection ~ 30000 13300
@@
 	1    0    0    -1
 $EndComp
+Text Notes 19500 7050 0    60   ~ 0
+WR+
+Text Notes 20100 9450 0    60   ~ 0
+RD+
+Wire Wire Line
+	8450 24100 8500 24100
+Connection ~ 8450 24300
+Wire Wire Line
+	10200 21000 10450 21000
+Wire Wire Line
+	10450 21000 10450 20550
+Wire Wire Line
+	10450 20550 9400 20550
+Wire Wire Line
+	9400 20550 9400 20400
+Wire Wire Line
+	9400 20400 4850 20400
+Wire Wire Line
+	4850 20400 4850 19500
+Connection ~ 4850 19500
+Wire Wire Line
+	10200 21000 10200 21550
+Wire Wire Line
+	15950 22150 15950 22850
+Text Notes 7850 6250 0    60   ~ 0
+A14
+Text Notes 7900 6900 0    60   ~ 0
+A15
+Text Notes 7900 6700 0    60   ~ 0
+port 0 Q4 - bit3
+Text Notes 7850 6050 0    60   ~ 0
+port 0 Q5 - bit2
+Text Notes 7850 6150 0    60   ~ 0
+port 1 Q5 - bit2
+Text Notes 9800 6100 0    60   ~ 0
+port D2
+Text Notes 9800 5750 0    60   ~ 0
+port D3
+Text Notes 6250 6800 0    60   ~ 0
+A15
+Text Notes 6250 6150 0    60   ~ 0
+A14
+Text Label 8050 7050 0    60   ~ 0
+GND
+Text Label 7950 7750 0    60   ~ 0
+GND
+Text Label 7950 8200 0    60   ~ 0
+GND
+Text Label 7950 8400 0    60   ~ 0
+GND
+Text Label 7950 8850 0    60   ~ 0
+GND
+Text Notes 9150 6200 0    60   ~ 0
+A19
+Text Notes 9150 6300 0    60   ~ 0
+A18
+Text Notes 9150 6400 0    60   ~ 0
+A17
+Text Notes 9150 6500 0    60   ~ 0
+A16
+Text Notes 8050 5600 0    60   ~ 0
+A15
+Text Notes 8050 5500 0    60   ~ 0
+A14
+Text Notes 10850 6900 0    60   ~ 0
+b0
+Text Notes 10850 6800 0    60   ~ 0
+b1
+Text Notes 10850 6700 0    60   ~ 0
+b2
+Text Notes 10850 6600 0    60   ~ 0
+b3
+Text Notes 10850 6500 0    60   ~ 0
+b4
+Text Notes 10850 6400 0    60   ~ 0
+b5
+Text Notes 10850 6300 0    60   ~ 0
+b6
+Text Notes 10850 6200 0    60   ~ 0
+b7
+Text Notes 10850 5300 0    60   ~ 0
+b0
+Text Notes 10850 5200 0    60   ~ 0
+b1
+Text Notes 10850 5100 0    60   ~ 0
+b2
+Text Notes 10850 5000 0    60   ~ 0
+b3
+Text Notes 10850 4900 0    60   ~ 0
+b4
+Text Notes 10850 4800 0    60   ~ 0
+b5
+Text Notes 10850 4700 0    60   ~ 0
+b6
+Text Notes 10850 4600 0    60   ~ 0
+b7
+Text Notes 7900 6800 0    60   ~ 0
+port 1 Q4 - bit3
+Text Notes 8050 5100 0    60   ~ 0
+A16
+Text Notes 8050 5000 0    60   ~ 0
+A16
+Text Notes 8050 5250 0    60   ~ 0
+A17
+Text Notes 8050 5350 0    60   ~ 0
+A17
+Text Notes 8050 4850 0    60   ~ 0
+A18
+Text Notes 8050 4750 0    60   ~ 0
+A18
+Text Notes 8050 4500 0    60   ~ 0
+A19
+Text Notes 8050 4600 0    60   ~ 0
+A19
+Wire Wire Line
+	7600 24100 8050 24100
 $EndSCHEMATC
