File: XC9500-IO/XC9500v1.sch (KiCad schematic (older format))
At the start: 112 parts, among them IC1 XC9572PC84, IC10 MCP23S08SO, IC11 MCP23S08SO, IC12 MCP23S08SO, IC13 MCP23S08SO, IC2 MCP23S08SO, IC3 MCP23S08SO, IC4 MCP23S08SO, IC5 MCP23S08SO, IC6 MCP23S08SO, IC7 MCP23S08SO, IC8 MCP23S08SO, IC9 MCP23S08SO, K1 CONN_3, P1 CONN_2, P10 XILINX CABLE2, P11 MCP_3_4, P12 MCP_5_6, P13 MCP_7_8, P14 MCP_9_10, P15 MCP_11_12, P19 S100_MALE, P2 EXTRN_SPI_1, P3 CONN_2, P4 CLK3, P5 EXTRN_SPI_2, P6 CONN_1, P7 CONN_1, P8 MCP_1_2, P9 CONN_7X2, SW1 DIPS_08, U1 74LS244, U10 74LS682N, U18 ^^74LS541, U2 74LVC245, U20 ^^74LS541, U21 74LVC245, U22 74LVC245, U24 74LVC245, U3 LM1086CS, U31 23LC1024, U34 LDO_REG_7805, U4 ^^LOGO1, U45 74LVC245, U5 74LVC1T45, U6 74LVC1T45, U7 74LVC1T45, U8 74LVC1T45, U9 M25P80

Commit message: XC9500-IO: SPI and chip-select pull-ups, INT3/INT4 select jumpers, decode jumper P20, BOM
Source: S100 XC9500 Ver1/backups/26-07-2015 2206 before ses (folder named before the autorouter session import; the .ses is not included).
Parts:
- removed P2: EXTRN_SPI_1, symbol CONN_6
- removed P5: EXTRN_SPI_2, symbol CONN_6
- added C30: 0.1 uF, symbol C
- added C31: 10 uF, symbol CP
- added P16: CONN_2, ~, symbol CONN_2
- added P17: INT3, ~, symbol CONN_3
- added P18: INT4, ~, symbol CONN_3
- added P2: EXTRN_SPI_1, symbol CONN_8
- added P5: EXTRN_SPI_2, symbol CONN_8
- added R12, R13, R14, R15, R16, R17, R19, R20, R21, R22, R23, R28, R30, R31, R32: 10K, symbol R
- renumbered K1 to P20
Connections:
- net labels added: EXTSPI_1_INT, EXTSPI_2_INT
- net labels removed: 3.3b
- wire segments 1231 -> 1300
Other:
- moved on the sheet: C21, C4, R7, R9

Commit message: XC9500-IO: routed board, add EXTERNAL MCP11/12 SPI header P21
Source: S100 XC9500 Ver1/backups/29-07-2015 1801. First routed layout (Specctra session imported).
Parts:
- added P21: ETRN SPI 11/12, symbol CONN_7X2
Connections:
- wire segments 1300 -> 1316
Other:
- note added: "External SPI interface Un-buffered\nTake over CS pins for MCP11 and MCP 12\ndont populate MCP11/12 if using this header"
- moved on the sheet: P1, P16, P3
Changed lines of the file:
@@
 Sheet 1 1
 Title "noname.sch"
-Date "25 jul 2015"
+Date "29 jul 2015"
 Rev ""
 Comp ""
@@
 Wire Wire Line
 	8250 3650 8350 3650
-Text Label 6900 5550 0    60   ~ 0
+Text Label 7600 5750 0    60   ~ 0
 V5.0temp
 Wire Wire Line
@@
 L CONN_2 P1
 U 1 1 55B2E100
-P 8300 5050
-F 0 "P1" V 8250 5050 40  0000 C CNN
-F 1 "CONN_2" V 8350 5050 40  0000 C CNN
-F 2 "~" H 8300 5050 60  0000 C CNN
-F 3 "~" H 8300 5050 60  0000 C CNN
-	1    8300 5050
+P 8950 5000
+F 0 "P1" V 8900 5000 40  0000 C CNN
+F 1 "CONN_2" V 9000 5000 40  0000 C CNN
+F 2 "~" H 8950 5000 60  0000 C CNN
+F 3 "~" H 8950 5000 60  0000 C CNN
+	1    8950 5000
 	1    0    0    -1
 $EndComp
@@
 L CONN_2 P3
 U 1 1 55B2E10D
-P 8300 5400
-F 0 "P3" V 8250 5400 40  0000 C CNN
-F 1 "CONN_2" V 8350 5400 40  0000 C CNN
-F 2 "~" H 8300 5400 60  0000 C CNN
-F 3 "~" H 8300 5400 60  0000 C CNN
-	1    8300 5400
+P 8950 5350
+F 0 "P3" V 8900 5350 40  0000 C CNN
+F 1 "CONN_2" V 9000 5350 40  0000 C CNN
+F 2 "~" H 8950 5350 60  0000 C CNN
+F 3 "~" H 8950 5350 60  0000 C CNN
+	1    8950 5350
 	1    0    0    -1
 $EndComp
@@
 	7550 4950 7950 4950
 Wire Wire Line
-	7550 5300 7950 5300
+	7550 5300 8050 5300
 Connection ~ 7550 4950
 Wire Wire Line
@@
 	7450 5500 7950 5500
 Wire Wire Line
-	7750 5150 7950 5150
+	7750 5150 8050 5150
 Wire Wire Line
 	7750 5150 7750 5500
@@
 	1000 16450 8050 16450
 Wire Notes Line
-	9500 32150 19400 32150
-Wire Notes Line
-	19400 32150 19400 11900
+	9500 32150 22650 32150
 Wire Notes Line
 	19400 11900 9500 11900
@@
 L CONN_2 P16
 U 1 1 55BA3051
-P 8200 27150
-F 0 "P16" V 8150 27150 40  0000 C CNN
-F 1 "CONN_2" V 8250 27150 40  0000 C CNN
-F 2 "~" H 8200 27150 60  0000 C CNN
-F 3 "~" H 8200 27150 60  0000 C CNN
-	1    8200 27150
+P 8450 27050
+F 0 "P16" V 8400 27050 40  0000 C CNN
+F 1 "CONN_2" V 8500 27050 40  0000 C CNN
+F 2 "~" H 8450 27050 60  0000 C CNN
+F 3 "~" H 8450 27050 60  0000 C CNN
+	1    8450 27050
 	1    0    0    -1
 $EndComp
@@
 	7750 26800 7750 27050
 Wire Wire Line
-	7750 27050 7850 27050
+	7750 27050 7900 27050
 Text Label 7700 27450 0    60   ~ 0
 V5.0temp
 Wire Wire Line
-	7850 27250 7600 27250
+	7600 27250 7900 27250
 Wire Wire Line
 	7600 27250 7600 27450
@@
 	1    0    0    -1
 $EndComp
+Text Label 21100 30450 0    60   ~ 0
+SPI_SCK
+Text Label 21100 30550 0    60   ~ 0
+SPI_SI
+Text Label 20100 30650 2    60   ~ 0
+SPI_S0
+Wire Notes Line
+	22650 32150 22650 26750
+Wire Notes Line
+	22650 26750 19400 26750
+Wire Notes Line
+	19400 26750 19400 11900
+Text Label 20100 30850 2    60   ~ 0
+MCP12_CS
+Text Label 20100 30750 2    60   ~ 0
+BOARD_RESET*
+Text Label 20100 30950 2    60   ~ 0
+V5.0
+Text Label 21100 30850 0    60   ~ 0
+MCP11_CS
+Text Label 21100 30950 0    60   ~ 0
+V5.0
+Text Label 20100 30350 2    60   ~ 0
+GND
+Text Label 21100 30350 0    60   ~ 0
+GND
+Text Label 20100 30550 2    60   ~ 0
+SPI_SI
+Text Label 21100 30650 0    60   ~ 0
+SPI_S0
+Text Label 20100 30450 2    60   ~ 0
+SPI_SCK
+Text Label 21100 30750 0    60   ~ 0
+BOARD_RESET*
+Wire Wire Line
+	21100 30350 21000 30350
+Wire Wire Line
+	21000 30450 21100 30450
+Wire Wire Line
+	21100 30550 21000 30550
+Wire Wire Line
+	21000 30650 21100 30650
+Wire Wire Line
+	21100 30750 21000 30750
+Wire Wire Line
+	21000 30850 21100 30850
+Wire Wire Line
+	20100 30350 20200 30350
+Wire Wire Line
+	20200 30450 20100 30450
+Wire Wire Line
+	20100 30550 20200 30550
+Wire Wire Line
+	20200 30650 20100 30650
+Wire Wire Line
+	20100 30750 20200 30750
+Wire Wire Line
+	20200 30850 20100 30850
+Text Notes 19100 29700 0    118  ~ 0
+External SPI interface Un-buffered\nTake over CS pins for MCP11 and MCP 12\ndont populate MCP11/12 if using this header
+Wire Wire Line
+	8050 5150 8050 5300
+Wire Wire Line
+	7900 27250 7900 27050
+$Comp
+L CONN_7X2 P21
+U 1 1 55B8D131
+P 20600 30650
+F 0 "P21" H 20600 31050 60  0000 C CNN
+F 1 "ETRN SPI 11/12" V 20600 30650 60  0000 C CNN
+F 2 "" H 20600 30650 60  0000 C CNN
+F 3 "" H 20600 30650 60  0000 C CNN
+	1    20600 30650
+	1    0    0    -1
+$EndComp
+Wire Wire Line
+	21100 30950 21000 30950
+Wire Wire Line
+	20200 30950 20100 30950
 $EndSCHEMATC

Commit message: XC9500-IO: schematic rev after the gerbers - U11 74LS682 for A5-A7, 12-way SW1, VI0* on the vector jumper
Source: S100 XC9500 Ver1 working folder (schematic and cache lib 13-08-2015, netlist and cmp 01-08-2015).
Parts:
- removed P1, P16, P3: CONN_2, ~, symbol CONN_2
- removed P9: CONN_7X2, symbol CONN_7X2
- removed SW1: DIPS_08, SWDIP8, symbol DIPS_08
- added C33: 0.1 uF, symbol C
- added P9: CONN_8X2, symbol CONN_8X2
- added SW1: DIPS_12, symbol DIPS_12
- added U11: 74LS682N, 20dip300, symbol 74LS682N
Connections:
- net labels added: VI0*b
- wire segments 1316 -> 1379
- no-connect marks 28 -> 29
Other:
- note added: "TOP ADDR\nA15\nA14\nA13\nA12\nA11\nA10\nA9\nA8\nA7\nA6\nA5"
- moved on the sheet: P20, U10
