File: Z80-CPU/v5/s100_Z80 V5.sch (KiCad schematic (older format))
At the start: 139 parts, among them IC1 XC9572PC84, K1 ROM LOCK, K17 EN_WAITS, K2 CONN_3, K3 SLAVE_CLR, P1 S100_MALE, P10 CONN_2, P11 CONN_6, P2 CONN_4X2, P3 CLK_CPU, P34 CONN_1, P35 CONN_1, P36 CONN_3X2, P4 CONN_2X2, P5 XILINX CABLE2, P6 MASTER_OSC, P7 NMI, P9 CONN_2, Q1 ^^NPN-SOT23, Q2 ^^NPN-SOT23, Q3 ^^NPN-SOT23, SW1 RESET, SW2 DIPS_08, SW3 DIPS_08, SW4 DIPS_08, U1 Z80, U10 74LS165, U11 74LS165, U12 74LVC573, U13 2732, U14 74LS682N, U15 74LS153, U16 74LS153, U17 74LS08, U19 74LS244, U2 74LVC573, U20 74LS244, U21 ^^74LS541, U22 74LVC573, U23 74LS02, U26 ^^LOGO1, U27 74LS139, U28 74LS00, U29 74LS273, U3 74LVC573, U30 74LS273, U31 74LS00, U32 74LS273, U33 74LS74, U34 74LS74, U36 74LS04, U37 74LS05, U39 74LS273, U4 74LS04, U45 74LS02, U48 LDO_REG_7805, U5 74LS157, U6 74LS157, U8 74LS157, U9 74LS165

Commit message: Z80-CPU v5: schematic and placement
Source: S100 Z80 version5/backups/28-12-2015 before ses
Newest file is 2015-12-27 18:14.
Parts:
- removed P11: CONN_6, symbol CONN_6
- removed P6: MASTER_OSC, ~, symbol CONN_3X2
- removed R20: 10k, symbol R
- added P11: CONN_5X2, symbol CONN_5X2
- added P6: CLK SEL, symbol CONN_2X2
- D1: value DONE -> ACTIVE
- D2: value DONE -> ROM
Connections:
- net labels added: CPLD_P45, CPLD_P53, CPLD_P56, CPLD_P57
- net labels removed: RD+
- wire segments 1355 -> 1364
Other:
- note added: "(aka RD+)"
- note added: "Board Reset Logic"
- note added: "D4 input"
- note added: "D5 input"
- note added: "D6 input"
- note added: "D7 input"
- note removed: "2 input AND"
- note removed: "Clave clear from CPLD - output"
- note removed: "WR+ output"
- note removed: "would come from\nSlave clear via CPLD"
- moved on the sheet: P7, U4D, U4E

Commit message: Z80-CPU v5: REV 5.0 gerbers, logo and final schematic
Source: S100 Z80 version5 (working folder): GERBERS, logo/, .sch, -cache.lib, .net, .cmp.
The routed board at gerber time was not kept separately; the only routed copy is the 2016-10-29 save in the next commit.
Parts:
- removed P10, P9: CONN_2, ~, symbol CONN_2
- removed U13: 2732, symbol 2732
- added P8: CONN_2, ~, symbol CONN_2
- added R20, R5: 1K, R3, symbol R
- added U13: 2764, symbol 2764
Connections:
- wire segments 1364 -> 1393
Other:
- note added: "2764 or 2732 EPROM\n2732 pin 1 = 2764 pin 3\n\nNote: with 2732 jumper P8 must be onnected for 5v power\n"
- moved on the sheet: P5, R10, R11, R12
