File: Z80-CPU/v5/s100_Z80 V5.kicad_pcb (KiCad board)
At the start: 2 copper layers, 254 x 134.6 mm, 139 parts, among them IC1 XC9572PC84, K1 ROM LOCK, K17 EN_WAITS, K2 CONN_3, K3 SLAVE_CLR, P1 S100_MALE, P10 CONN_2, P11 CONN_6, P2 CONN_4X2, P3 CLK_CPU, P34 CONN_1, P35 CONN_1, P36 CONN_3X2, P4 CONN_2X2, P5 XILINX CABLE2, P6 MASTER_OSC, P7 NMI, P9 CONN_2, Q1 ^^NPN-SOT23, Q2 ^^NPN-SOT23, Q3 ^^NPN-SOT23, SW1 RESET, SW2 DIPS_08, SW3 DIPS_08, SW4 DIPS_08, U1 Z80, U10 74LS165, U11 74LS165, U12 74LVC573, U13 2732, U14 74LS682N, U15 74LS153, U16 74LS153, U17 74LS08, U19 74LS244, U2 74LVC573, U20 74LS244, U21 ^^74LS541, U22 74LVC573, U23 74LS02, U26 ^^LOGO1, U27 74LS139, U28 74LS00, U29 74LS273, U3 74LVC573, U30 74LS273, U31 74LS00, U32 74LS273, U33 74LS74, U34 74LS74, U36 74LS04, U37 74LS05, U39 74LS273, U4 74LS04, U45 74LS02, U48 LDO_REG_7805, U5 74LS157, U6 74LS157, U8 74LS157, U9 74LS165

Commit message: Z80-CPU v5: schematic and placement
Source: S100 Z80 version5/backups/28-12-2015 before ses
Newest file is 2015-12-27 18:14.
Parts:
- removed R20: 10k, R3
- D1: value DONE -> ACTIVE
- D2: value DONE -> ROM
- P11: value CONN_6 -> CONN_5X2; footprint PIN_ARRAY_6X1 -> PIN_ARRAY_5X2
- P6: value MASTER_OSC -> CLK SEL; footprint PIN_ARRAY_3X2 -> PIN_ARRAY_2X2
- moved R19 155.0 mm to (73.8, 39.4), turned to 90 degrees
- moved SW1 136.1 mm to (70.2, 29.3)
- moved P7 81.4 mm to (187.3, 99.1)
- moved U28 74.0 mm to (245.1, 97.9)
- moved C14 74.0 mm to (232.4, 97.9)
- moved P2 65.0 mm to (254.1, 106.9), turned to 0 degrees
- moved P36 59.5 mm to (242.4, 106.9), turned to 0 degrees
- moved U8 54.4 mm to (209.3, 66.3)
- moved C27 54.4 mm to (195.6, 66.3)
- moved P4 47.2 mm to (232.3, 107.0), turned to 0 degrees
- moved C46 45.7 mm to (158.8, 33.1)
- moved U36 45.7 mm to (171.4, 33.1)
- moved C8 44.0 mm to (158.8, 50.4)
- moved U39 44.0 mm to (175.3, 50.8)
- moved C2 39.5 mm to (85.1, 78.7)
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Connections:
- IC1 pad 10: (no net) -> /CPLD_CLKout1
- IC1 pad 12: (no net) -> /CPLD_CLKout2
- IC1 pad 15: (no net) -> /CPLD_P15
- IC1 pad 23: (no net) -> /CPLD_P23
- IC1 pad 45: (no net) -> /CPLD_P45
- IC1 pad 52: (no net) -> /CPLD_P52
- IC1 pad 53: (no net) -> /CPLD_P53
- IC1 pad 56: (no net) -> /CPLD_P56
- IC1 pad 57: (no net) -> /CPLD_P57
- K17 pad 3: (no net) -> /PU1K-waits
- P11 pad 1: GND -> /CPLD_P75
- P11 pad 2: /CPLD_P75 -> GND
- P11 pad 4: /CPLD_P4 -> /CPLD_P15
- P11 pad 5: /CPLD_P77 -> /CPLD_P4
- P11 pad 6: /CPLD_P3 -> /CPLD_P23
- RR5 pad 10: (no net) -> /PU1K-waits
- U1 pad 10: /D6 -> /CPLD_P53
- U1 pad 13: /D7 -> /CPLD_P57
- U1 pad 7: /D4 -> /CPLD_P45
- U1 pad 9: /D5 -> /CPLD_P56
- U13 pad 14: /D4 -> /CPLD_P45
- U13 pad 15: /D5 -> /CPLD_P56
- U13 pad 16: /D6 -> /CPLD_P53
- U13 pad 17: /D7 -> /CPLD_P57
- U19 pad 2: /D7 -> /CPLD_P57
- U19 pad 4: /D6 -> /CPLD_P53
- U19 pad 6: /D5 -> /CPLD_P56
- U19 pad 8: /D4 -> /CPLD_P45
- U20 pad 12: /D4 -> /CPLD_P45
- U20 pad 14: /D5 -> /CPLD_P56
- U20 pad 16: /D6 -> /CPLD_P53
- U20 pad 18: /D7 -> /CPLD_P57
- U21 pad 6: /CLK_CPUneg -> /CPLD_CLKout2
- U21 pad 7: (no net) -> /CPLD_CLKout1
- U29 pad 3: /D7 -> /CPLD_P57
- U29 pad 4: /D6 -> /CPLD_P53
- U29 pad 7: /D5 -> /CPLD_P56
- U29 pad 8: /D4 -> /CPLD_P45
- U30 pad 3: /D7 -> /CPLD_P57
- U30 pad 4: /D6 -> /CPLD_P53
- U30 pad 7: /D5 -> /CPLD_P56
- U30 pad 8: /D4 -> /CPLD_P45
- U32 pad 3: /D7 -> /CPLD_P57
- U32 pad 4: /D6 -> /CPLD_P53
- U32 pad 7: /D5 -> /CPLD_P56
- U32 pad 8: /D4 -> /CPLD_P45
- U39 pad 3: /D7 -> /CPLD_P57
- U39 pad 4: /D6 -> /CPLD_P53
- U39 pad 7: /D5 -> /CPLD_P56
- U39 pad 8: /D4 -> /CPLD_P45
Routing:
- net N-00000188: track 0.00 -> 4.40 mm, vias 0 -> 1
- net N-00000183: track 0.00 -> 4.32 mm, vias 0 -> 1
- net N-00000187: track 0.00 -> 4.25 mm, vias 0 -> 1
- net N-00000184: track 0.00 -> 4.25 mm, vias 0 -> 1
- net N-00000182: track 0.00 -> 4.25 mm, vias 0 -> 1
- net N-00000181: track 0.00 -> 4.14 mm, vias 0 -> 1
Other:
- net class Default: trace_width 0.25 -> 0.23
- net class gnd: trace_width 0.25 -> 0.23

Commit message: Z80-CPU v5: routed trial
Source: S100 Z80 version5/backups/29-12-2015 morning
Routing:
- net GND: track 0.00 -> 1646.8 mm, vias 0 -> 9
- net VCC: track 0.00 -> 1153.9 mm, vias 0 -> 2
- net /CPLD_P43: track 0.00 -> 429.2 mm, vias 0 -> 6
- net /CPLD_P36: track 0.00 -> 405.3 mm, vias 0 -> 5
- net /CPLD_P7: track 0.00 -> 390.0 mm, vias 0 -> 6
- net /CPLD_P21: track 0.00 -> 387.1 mm
- net /CPLD_P2: track 0.00 -> 380.1 mm, vias 0 -> 7
- net /CPLD_P82: track 0.00 -> 367.0 mm, vias 0 -> 4
- net /CPLD_P71: track 0.00 -> 366.9 mm, vias 0 -> 2
- net /CPLD_P31: track 0.00 -> 362.1 mm, vias 0 -> 5
- net /CPLD_P13: track 0.00 -> 358.7 mm, vias 0 -> 2
- net /CPLD_P24: track 0.00 -> 352.9 mm, vias 0 -> 6
- net /CPLD_P18: track 0.00 -> 348.4 mm, vias 0 -> 3
- net /CPLD_P32: track 0.00 -> 347.2 mm, vias 0 -> 6
- net /CPLD_P56: track 0.00 -> 334.7 mm, vias 0 -> 2
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
Commit message: Z80-CPU v5: schematic and placement before routing
Source: S100 Z80 version5/backups/30-12-2015 before ses
Newest file is 2015-12-29 12:45.
Routing:
- net GND: track 1646.8 -> 0.00 mm, vias 9 -> 0
- net VCC: track 1153.9 -> 23.0 mm, vias 2 -> 0
- net /CPLD_P43: track 429.2 -> 0.00 mm, vias 6 -> 0
- net /CPLD_P36: track 405.3 -> 0.00 mm, vias 5 -> 0
- net /CPLD_P7: track 390.0 -> 0.00 mm, vias 6 -> 0
- net /CPLD_P21: track 387.1 -> 0.00 mm
- net /CPLD_P2: track 380.1 -> 0.00 mm, vias 7 -> 0
- net /CPLD_P82: track 367.0 -> 0.00 mm, vias 4 -> 0
- net /CPLD_P71: track 366.9 -> 0.00 mm, vias 2 -> 0
- net /CPLD_P31: track 362.1 -> 0.00 mm, vias 5 -> 0
- net /CPLD_P13: track 358.7 -> 0.00 mm, vias 2 -> 0
- net /CPLD_P24: track 352.9 -> 0.00 mm, vias 6 -> 0
- net /CPLD_P18: track 348.4 -> 0.00 mm, vias 3 -> 0
- net /CPLD_P32: track 347.2 -> 0.00 mm, vias 6 -> 0
- net /CPLD_P56: track 334.7 -> 0.00 mm, vias 2 -> 0
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
Commit message: Z80-CPU v5: routed board, CLK_OSC traces widened to 0.35 mm
Source: S100 Z80 version5/s100_Z80 V5.kicad_pcb (working folder, saved 2016-10-29). The only surviving routed copy of the v5 board; it also changes the bottom text to '(c) 2016'.
Parts:
- removed P10, P9: CONN_2, PIN_ARRAY_2X1
- added P8: CONN_2, PIN_ARRAY_2X1, F.Cu at (155.9, 61.5)
- added R20: 1K, R3, F.Cu at (155.2, 93.8)
- added R5: 1K, R3, F.Cu at (158.5, 59.1)
- U13: value 2732 -> 2764; footprint ^^DIL24-6 -> DIP-28__600_ELL
- moved C6 7.12 mm to (148.9, 73.9)
- moved U13 2.57 mm to (171.1, 73.6)
- moved R2 0.56 mm to (227.3, 37.3), turned to 270 degrees
- moved R9 0.33 mm to (243.0, 37.2), turned to 270 degrees
- moved U26 0.24 mm to (230.3, 143.6)
- moved R6 0.22 mm to (235.2, 37.3), turned to 270 degrees
Connections:
- IC1 pad 22: /V5.0temp -> VCC
- IC1 pad 38: /V5.0temp -> VCC
- IC1 pad 64: /V5.0temp -> VCC
- IC1 pad 73: /V5.0temp -> VCC
- IC1 pad 78: /V5.0temp -> VCC
- U13 pad 1: /CPLD_P71 -> N-00000154
- U13 pad 10: /CPLD_P32 -> /CPLD_P80
- U13 pad 11: /CPLD_P31 -> /CPLD_P33
- U13 pad 12: GND -> /CPLD_P32
- U13 pad 13: /CPLD_P24 -> /CPLD_P31
- U13 pad 14: /CPLD_P45 -> GND
- U13 pad 15: /CPLD_P56 -> /CPLD_P24
- U13 pad 16: /CPLD_P53 -> /CPLD_P45
- U13 pad 17: /CPLD_P57 -> /CPLD_P56
- U13 pad 18: GND -> /CPLD_P53
- U13 pad 19: /bA10 -> /CPLD_P57
- U13 pad 2: /CPLD_P36 -> /CPLD_P34
- U13 pad 20: /27_ROM_OE -> GND
- U13 pad 21: /bA11 -> /bA10
- U13 pad 22: /bA9 -> /27_ROM_OE
- U13 pad 23: /bA8 -> /bA11
- U13 pad 24: VCC -> /bA9
- U13 pad 3: /CPLD_P43 -> /CPLD_P71
- U13 pad 4: /CPLD_P2 -> /CPLD_P36
- U13 pad 5: /CPLD_P7 -> /CPLD_P43
- U13 pad 6: /CPLD_P82 -> /CPLD_P2
- U13 pad 7: /CPLD_P83 -> /CPLD_P7
- U13 pad 8: /CPLD_P80 -> /CPLD_P82
- U13 pad 9: /CPLD_P33 -> /CPLD_P83
Routing:
- net GND: track 0.00 -> 1883.1 mm, vias 0 -> 22
- net VCC: track 23.0 -> 1178.5 mm, vias 0 -> 3
- net /CPLD_P82: track 0.00 -> 411.6 mm, vias 0 -> 8
- net /CPLD_P7: track 0.00 -> 408.4 mm, vias 0 -> 13
- net /CPLD_P43: track 0.00 -> 399.2 mm, vias 0 -> 4
- net /CPLD_P2: track 0.00 -> 382.7 mm, vias 0 -> 5
- net /CPLD_P36: track 0.00 -> 373.4 mm, vias 0 -> 6
- net /CPLD_P56: track 0.00 -> 362.1 mm, vias 0 -> 1
- net /CPLD_P71: track 0.00 -> 359.4 mm, vias 0 -> 6
- net /CPLD_P19: track 0.00 -> 358.3 mm, vias 0 -> 4
- net /CPLD_P57: track 0.00 -> 351.5 mm, vias 0 -> 2
- net /CPLD_P32: track 0.00 -> 346.9 mm, vias 0 -> 5
- net /CPLD_P18: track 0.00 -> 346.9 mm, vias 0 -> 3
- net /CPLD_P13: track 0.00 -> 346.6 mm, vias 0 -> 2
- net /CPLD_P24: track 0.00 -> 342.6 mm, vias 0 -> 6
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- added copper zone on B.Cu, net GND
- added copper zone on F.Cu, net GND
Other:
- board text added: "I/O WAIT"
- board text added: "RAM WAIT"
- board text added: "ROM SELECT"
- board text added: "U13 2764/2732"
- board text added: "Z80 CPU © 2016 A Burrows"
- board text removed: "IO WAIT"
- board text removed: "MEM WAIT"
- board text removed: "ROM READ"
- board text removed: "Z80 CPU © 2015 A Burrows"
